File: power/power.sch (KiCad schematic (older format))
At the start: 32 parts

Commit message: Removed PGA+RMS, added preheat relay
Parts:
- removed C?: C, symbol C
- removed C?: 2.2uF, symbol C
- removed P?: CONN_02X03, symbol CONN_02X03
- removed U?: LTC1966, symbol LTC1966
- removed U?: LTC6910, symbol LTC6910
- added K2: RELAY_2RT, symbol RELAY_2RT
- added P3: CONN_02X04, symbol CONN_02X04
- added Q2: BC636, TO92, symbol BC636
- added R2: R, symbol R
- gave numbers to parts that had none: 27
Connections:
- net labels added: MASTER_RELAY, PREHEAT_RELAY
- net labels removed: ISENSE_VRMS, PASS_RELAY, SGA_G0, SGA_G1, SGA_G2
- wire segments 139 -> 120
- no-connect marks 2 -> 9
Other:
- note added: "CONNECTORS"
- note added: "CROSSOVER SENSE"
- note added: "CURRENT SENSE"
- note added: "LOAD CONTORL"
- note added: "MASTER"
- note added: "POWER SUPPLY"
- note added: "PREHEAT"
- note removed: "Capacitor\nfor averaging"

Commit message: SPST relays, filled in many values
Parts:
- removed C5: CP2, symbol CP2
- removed K1, K2: RELAY_2RT, symbol RELAY_2RT
- removed Q1, Q2: BC636, TO92, symbol BC636
- added K1, K2, K3: RELAY_SPST, symbol RELAY_SPST
- added Q1, Q2, Q3: BC817-40, SOT-23, symbol BC817-40
- added R10: 390R, symbol R
- C1: value CP2 -> 220uF
- C2: value C -> 22nF
- C3: value C -> 0.33uF
- C4: value C -> 0.1uF
- C6: value C -> 1nF
- C7: value C -> 100nF
- C9: value C -> 1uF
- R1, R2: value R -> 390R
- R4: value R -> 47R
- R6: value R -> 1k
- R7: value R -> 30k
- R8: value R -> 150R
- R9: value R -> 15k
- U1: Farnell (none) -> 1696994
Connections:
- wire segments 120 -> 125
- no-connect marks 9 -> 3
Other:
- note added: "LOAD CONTROL"
- note removed: "LOAD CONTORL"

Commit message: P sch: up2date connector, dbl winding xformer
Parts:
- removed P3: CONN_02X04, symbol CONN_02X04
- removed T1: 240-6VAC, symbol TRANSFO
- added P?: CONTROL, symbol CONN_02X04
- added T?: 240-2x6VAC, symbol TRANSFO2
Connections:
- net labels added: 6VAC_SENSE, LV_RECTIFIED
- net labels removed: HV_RECTIFIED
- wire segments 125 -> 129

Commit message: P sch: filled in most component part #s
Parts:
- removed R7: 30k, symbol R
- added R? (x2): 15k, symbol R
- C1: Farnell (none) -> 2346447
- C2: renamed from C3; Farnell (none) -> 1759153
- C3: renamed from C4; Farnell (none) -> 1759166
- C4: renamed from C9; Farnell (none) -> 2320857
- C5: renamed from C2; Farnell (none) -> 2057310
- C6: Farnell (none) -> 1759226
- C7, C8: Farnell (none) -> 1759166
- R1: renamed from R10; Farnell (none) -> 2331790
- R10: renamed from R5; value 210R -> 220R; Farnell (none) -> 2331787
- R2: renamed from R1; Farnell (none) -> 2331790
- R3: renamed from R2; Farnell (none) -> 2331790
- R4: renamed from R6; value 1k -> 1k5; Farnell (none) -> 2331798
- R6: renamed from R3; value 360R -> 390R; Farnell (none) -> 2331790
- R7: renamed from R8; value 150R -> 220R; Farnell (none) -> 2331787
- R8: renamed from R9; Farnell (none) -> 2331812
- R9: renamed from R4; Farnell (none) -> 1887414
- U2: value MOC3020 -> MOC3023; Farnell (none) -> 2322550
- U4: Farnell (none) -> 1791411
- gave numbers to parts that had none: 2
Connections:
- wire segments 129 -> 132
Other:
- note added: "56mV/A version:\nACS710KLATR-12CB-T"
- note added: "Sets bandwidth with\ninternal filter R"
Changed lines of the file:
@@
 F 2 "" H 5388 1850 30  0000 C CNN
 F 3 "" H 5350 2000 60  0000 C CNN
+F 4 "2346447" H 5350 2000 60  0001 C CNN "Farnell"
 	1    5350 2000
 	1    0    0    -1
@@
 LV_RECTIFIED
 $Comp
-L C C3
+L C C2
 U 1 1 54E4FD5B
 P 1650 3450
-F 0 "C3" H 1700 3550 50  0000 L CNN
+F 0 "C2" H 1700 3550 50  0000 L CNN
 F 1 "0.33uF" H 1700 3350 50  0000 L CNN
 F 2 "" H 1688 3300 30  0000 C CNN
 F 3 "" H 1650 3450 60  0000 C CNN
+F 4 "1759153" H 1650 3450 60  0001 C CNN "Farnell"
 	1    1650 3450
 	1    0    0    -1
 $EndComp
 $Comp
-L C C4
+L C C3
 U 1 1 54E4FD91
 P 2800 3450
-F 0 "C4" H 2850 3550 50  0000 L CNN
+F 0 "C3" H 2850 3550 50  0000 L CNN
 F 1 "0.1uF" H 2850 3350 50  0000 L CNN
 F 2 "" H 2838 3300 30  0000 C CNN
 F 3 "" H 2800 3450 60  0000 C CNN
+F 4 "1759166" H 2800 3450 60  0001 C CNN "Farnell"
 	1    2800 3450
 	1    0    0    -1
@@
 $EndComp
 $Comp
-L R R6
-U 1 1 54E5103B
-P 4400 3800
-F 0 "R6" V 4480 3800 50  0000 C CNN
-F 1 "1k" V 4407 3801 50  0000 C CNN
-F 2 "" V 4330 3800 30  0000 C CNN
-F 3 "" H 4400 3800 30  0000 C CNN
-	1    4400 3800
-	1    0    0    -1
-$EndComp
-$Comp
-L R R8
+L R R7
 U 1 1 54E510B7
 P 4400 4500
-F 0 "R8" V 4480 4500 50  0000 C CNN
-F 1 "150R" V 4407 4501 50  0000 C CNN
+F 0 "R7" V 4480 4500 50  0000 C CNN
+F 1 "220R" V 4407 4501 50  0000 C CNN
 F 2 "" V 4330 4500 30  0000 C CNN
 F 3 "" H 4400 4500 30  0000 C CNN
+F 4 "2331787" H 4400 4500 60  0001 C CNN "Farnell"
 	1    4400 4500
 	1    0    0    -1
@@
 $EndComp
 $Comp
-L C C9
+L C C4
 U 1 1 54E5148F
 P 4750 4100
-F 0 "C9" V 4800 4150 50  0000 L CNN
+F 0 "C4" V 4800 4150 50  0000 L CNN
 F 1 "1uF" V 4800 3900 50  0000 L CNN
 F 2 "" H 4788 3950 30  0000 C CNN
 F 3 "" H 4750 4100 60  0000 C CNN
+F 4 "2320857" H 4750 4100 60  0001 C CNN "Farnell"
 	1    4750 4100
 	0    1    1    0
 $EndComp
 $Comp
-L R R7
-U 1 1 54E51AE5
-P 5050 3800
-F 0 "R7" V 5130 3800 50  0000 C CNN
-F 1 "30k" V 5057 3801 50  0000 C CNN
-F 2 "" V 4980 3800 30  0000 C CNN
-F 3 "" H 5050 3800 30  0000 C CNN
-	1    5050 3800
-	1    0    0    -1
-$EndComp
-$Comp
-L R R9
+L R R8
 U 1 1 54E51B51
 P 5050 4500
-F 0 "R9" V 5130 4500 50  0000 C CNN
+F 0 "R8" V 5130 4500 50  0000 C CNN
 F 1 "15k" V 5057 4501 50  0000 C CNN
 F 2 "" V 4980 4500 30  0000 C CNN
 F 3 "" H 5050 4500 30  0000 C CNN
+F 4 "2331812" H 5050 4500 60  0001 C CNN "Farnell"
 	1    5050 4500
 	1    0    0    -1
@@
 L +5V #PWR09
 U 1 1 54E524D3
-P 5050 3500
-F 0 "#PWR09" H 5050 3350 60  0001 C CNN
-F 1 "+5V" H 5050 3640 60  0000 C CNN
-F 2 "" H 5050 3500 60  0000 C CNN
-F 3 "" H 5050 3500 60  0000 C CNN
-	1    5050 3500
+P 5250 3500
+F 0 "#PWR09" H 5250 3350 60  0001 C CNN
+F 1 "+5V" H 5250 3640 60  0000 C CNN
+F 2 "" H 5250 3500 60  0000 C CNN
+F 3 "" H 5250 3500 60  0000 C CNN
+	1    5250 3500
 	1    0    0    -1
 $EndComp
@@
 P 8100 4450
 F 0 "U2" H 8300 4750 60  0000 C CNN
-F 1 "MOC3020" H 8050 4150 60  0000 C CNN
+F 1 "MOC3023" H 8050 4150 60  0000 C CNN
 F 2 "" H 8100 4450 60  0000 C CNN
 F 3 "" H 8100 4450 60  0000 C CNN
+F 4 "2322550" H 8100 4450 60  0001 C CNN "Farnell"
 	1    8100 4450
 	1    0    0    -1
 $EndComp
 $Comp
-L R R3
+L R R6
 U 1 1 54E52E94
 P 9150 4250
-F 0 "R3" V 9230 4250 50  0000 C CNN
-F 1 "360R" V 9050 4250 50  0000 C CNN
+F 0 "R6" V 9230 4250 50  0000 C CNN
+F 1 "390R" V 9050 4250 50  0000 C CNN
 F 2 "" V 9080 4250 30  0000 C CNN
 F 3 "" H 9150 4250 30  0000 C CNN
+F 4 "2331790" H 9150 4250 60  0001 C CNN "Farnell"
 	1    9150 4250
 	0    1    1    0
@@
 MAINS_LIVE
 $Comp
-L R R4
+L R R9
 U 1 1 54E5366C
 P 10550 4750
-F 0 "R4" V 10630 4750 50  0000 C CNN
+F 0 "R9" V 10630 4750 50  0000 C CNN
 F 1 "47R" V 10557 4751 50  0000 C CNN
 F 2 "" V 10480 4750 30  0000 C CNN
 F 3 "" H 10550 4750 30  0000 C CNN
+F 4 "1887414" H 10550 4750 60  0001 C CNN "Farnell"
 	1    10550 4750
 	1    0    0    -1
 $EndComp
 $Comp
-L C C2
+L C C5
 U 1 1 54E536C9
 P 10550 4250
-F 0 "C2" H 10600 4350 50  0000 L CNN
+F 0 "C5" H 10600 4350 50  0000 L CNN
 F 1 "22nF" H 10600 4150 50  0000 L CNN
 F 2 "" H 10588 4100 30  0000 C CNN
 F 3 "" H 10550 4250 60  0000 C CNN
+F 4 "2057310" H 10550 4250 60  0001 C CNN "Farnell"
 	1    10550 4250
 	1    0    0    -1
@@
 TRIAC_TRIG
 $Comp
-L R R5
+L R R10
 U 1 1 54E53E1C
 P 7250 4800
-F 0 "R5" V 7330 4800 50  0000 C CNN
-F 1 "210R" V 7150 4800 50  0000 C CNN
+F 0 "R10" V 7330 4800 50  0000 C CNN
+F 1 "220R" V 7150 4800 50  0000 C CNN
 F 2 "" V 7180 4800 30  0000 C CNN
 F 3 "" H 7250 4800 30  0000 C CNN
+F 4 "2331787" H 7250 4800 60  0001 C CNN "Farnell"
 	1    7250 4800
 	1    0    0    -1
@@
 $EndComp
 $Comp
-L R R1
+L R R2
 U 1 1 54E5F195
 P 7350 1800
-F 0 "R1" V 7430 1800 50  0000 C CNN
+F 0 "R2" V 7430 1800 50  0000 C CNN
 F 1 "390R" V 7357 1801 50  0000 C CNN
 F 2 "" V 7280 1800 30  0000 C CNN
 F 3 "" H 7350 1800 30  0000 C CNN
+F 4 "2331790" H 7350 1800 60  0001 C CNN "Farnell"
 	1    7350 1800
 	0    1    1    0
@@
 F 2 "" H 6638 6800 30  0000 C CNN
 F 3 "" H 6600 6950 60  0000 C CNN
+F 4 "1759166" H 6600 6950 60  0001 C CNN "Farnell"
 	1    6600 6950
 	1    0    0    -1
@@
 P 6350 6950
 F 0 "C7" H 6400 7050 50  0000 L CNN
-F 1 "100nF" H 6100 6850 50  0000 L CNN
+F 1 "100nF" H 6050 6850 50  0000 L CNN
 F 2 "" H 6388 6800 30  0000 C CNN
 F 3 "" H 6350 6950 60  0000 C CNN
+F 4 "1759166" H 6350 6950 60  0001 C CNN "Farnell"
 	1    6350 6950
 	1    0    0    -1
@@
 F 2 "" H 5688 6800 30  0000 C CNN
 F 3 "" H 5650 6950 60  0000 C CNN
+F 4 "1759226" H 5650 6950 60  0001 C CNN "Farnell"
 	1    5650 6950
 	1    0    0    -1
@@
 F 2 "" H 5750 7000 60  0000 C CNN
 F 3 "" H 5750 7000 60  0000 C CNN
+F 4 "1791411" H 4750 6450 60  0001 C CNN "Farnell"
 	1    4750 6450
 	1    0    0    -1
@@
 $EndComp
 $Comp
-L R R2
+L R R3
 U 1 1 54E9E5AF
 P 7400 2850
-F 0 "R2" V 7480 2850 50  0000 C CNN
+F 0 "R3" V 7480 2850 50  0000 C CNN
 F 1 "390R" V 7407 2851 50  0000 C CNN
 F 2 "" V 7330 2850 30  0000 C CNN
 F 3 "" H 7400 2850 30  0000 C CNN
+F 4 "2331790" H 7400 2850 60  0001 C CNN "Farnell"
 	1    7400 2850
 	0    1    1    0
@@
 $EndComp
 $Comp
-L R R10
+L R R1
 U 1 1 54E81E83
 P 7350 1050
-F 0 "R10" V 7430 1050 50  0000 C CNN
+F 0 "R1" V 7430 1050 50  0000 C CNN
 F 1 "390R" V 7357 1051 50  0000 C CNN
 F 2 "" V 7280 1050 30  0000 C CNN
 F 3 "" H 7350 1050 30  0000 C CNN
+F 4 "2331790" H 7350 1050 60  0001 C CNN "Farnell"
 	1    7350 1050
 	0    1    1    0
@@
 $EndComp
 $Comp
-L CONN_02X04 P?
+L CONN_02X04 P3
 U 1 1 54E909DD
 P 1600 7100
-F 0 "P?" H 1600 7350 50  0000 C CNN
+F 0 "P3" H 1600 7350 50  0000 C CNN
 F 1 "CONTROL" H 1600 6850 50  0000 C CNN
 F 2 "" H 1600 5900 60  0000 C CNN
@@
 $EndComp
 $Comp
-L TRANSFO2 T?
+L TRANSFO2 T1
 U 1 1 54E9209B
 P 1800 1300
-F 0 "T?" H 1800 1800 50  0000 C CNN
+F 0 "T1" H 1800 1800 50  0000 C CNN
 F 1 "240-2x6VAC" H 1800 800 50  0000 C CNN
 F 2 "" H 1800 1300 60  0000 C CNN
@@
 $EndComp
 $Comp
-L GND #PWR?
+L GND #PWR028
 U 1 1 54E976CC
 P 2350 1800
-F 0 "#PWR?" H 2350 1550 60  0001 C CNN
+F 0 "#PWR028" H 2350 1550 60  0001 C CNN
 F 1 "GND" H 2350 1650 60  0000 C CNN
 F 2 "" H 2350 1800 60  0000 C CNN
@@
 Text GLabel 4200 3500 0    60   Input ~ 0
 6VAC_SENSE
+Text Notes 4300 7100 0    60   ~ 0
+56mV/A version:\nACS710KLATR-12CB-T
+$Comp
+L R R?
+U 1 1 54E9C1CA
+P 5050 3800
+F 0 "R?" V 4950 3800 50  0000 C CNN
+F 1 "15k" V 5057 3801 50  0000 C CNN
+F 2 "" V 4980 3800 30  0000 C CNN
+F 3 "" H 5050 3800 30  0000 C CNN
+F 4 "2331812" H 5050 3800 60  0001 C CNN "Farnell"
+	1    5050 3800
+	1    0    0    -1
+$EndComp
+$Comp
+L R R?
+U 1 1 54E9C2F3
+P 5250 3800
+F 0 "R?" V 5350 3800 50  0000 C CNN
+F 1 "15k" V 5257 3801 50  0000 C CNN
+F 2 "" V 5180 3800 30  0000 C CNN
+F 3 "" H 5250 3800 30  0000 C CNN
+F 4 "2331812" H 5250 3800 60  0001 C CNN "Farnell"
+	1    5250 3800
+	1    0    0    -1
+$EndComp
+$Comp
+L R R4
+U 1 1 54E5103B
+P 4400 3800
+F 0 "R4" V 4480 3800 50  0000 C CNN
+F 1 "1k5" V 4407 3801 50  0000 C CNN
+F 2 "" V 4330 3800 30  0000 C CNN
+F 3 "" H 4400 3800 30  0000 C CNN
+F 4 "2331798" H 4400 3800 60  0001 C CNN "Farnell"
+	1    4400 3800
+	1    0    0    -1
+$EndComp
+Text Notes 5750 7750 0    60   ~ 0
+Sets bandwidth with\ninternal filter R
 Wire Wire Line
 	1300 1100 1400 1100
@@
 	5050 4200 5350 4200
 Connection ~ 5050 4200
-Wire Wire Line
-	5050 3500 5050 3550
 Wire Wire Line
 	8700 4250 8900 4250
@@
 Wire Wire Line
 	2200 900  4450 900
+Wire Wire Line
+	5050 3550 5150 3550
+Wire Wire Line
+	5150 3550 5150 4050
+Wire Wire Line
+	5150 4050 5250 4050
+Wire Wire Line
+	5250 3550 5250 3500
+Wire Notes Line
+	6050 7000 6050 7550
+Wire Notes Line
+	6050 7000 6300 7000
+Wire Notes Line
+	6300 7000 6300 7100
+Wire Notes Line
+	6300 7100 6050 7100
 $EndSCHEMATC

Commit message: P sch: switcher PSU + tiny xover sense xformer
Parts:
- removed C1: 220uF, symbol CP2
- removed C2: 0.33uF, symbol C
- removed C3: 0.1uF, symbol C
- removed C4: 1uF, symbol C
- removed D1: BRIDGE, symbol BRIDGE
- removed R7: 220R, symbol R
- removed R8, R? (x2): 15k, symbol R
- removed T1: 240-2x6VAC, symbol TRANSFO2
- removed U1: 7805, symbol 7805
- added R2, R6: 10k, symbol R
- added R5: 3k3, symbol R
- added T1: 240VAC:6VAC 1VA, symbol TRANSFO
- added U1: VTX214, symbol VTX214
- added U?: AD813, symbol AD813
- R4: value 1k5 -> 10k; Farnell 2331798 -> 1887308
- renumbered C5 to C1, C6 to C2, C7 to C3, C8 to C4, R2 to R3, R3 to R7, R6 to R8, U2 to U3, U3 to U4, U4 to U5
Connections:
- net labels removed: 6VAC_SENSE, LV_RECTIFIED
- wire segments 132 -> 124
Other:
- note added: "+6VAC (RMS)"
- note added: "2.5VDC"
- note added: "2.5VDC +\n1.4VAC_RMS"
- note added: "5V 3W\nVTX-214-003-105"
- note added: "MAGIC BOX"
- note added: "MASTER LIVE"
- note added: "MASTER NEUTRAL"
- note added: "POWER SUPPLY & CROSSOVER SENSE"
- note added: "TODO: pick a decent opamp/comparator"
- note removed: "6VAC+"
- note removed: "6VAC-"
- note removed: "CROSSOVER SENSE"
- note removed: "MASTER"
- note removed: "POWER SUPPLY"

Commit message: Psch: crossover MOC, ds18b20, ERC
* Changed MOC chip to one with builtin crossover, removed crossover sensing
  circuit.
* Added DS18B20 temperature sensor (intended for mounting to the triac
  heatsink) on the pin previously used for crossover sense.
* Minor changes around the PSU area to make ERC pass.
Parts:
- removed R2, R4, R6: 10k, symbol R
- removed R5: 3k3, symbol R
- removed T1: 240VAC:6VAC 1VA, symbol TRANSFO
- removed U?: AD813, symbol AD813
- added F1: 100mA, symbol FUSE
- added F2: 13A, symbol FUSE
- added U5: DS18B20, symbol DS18B20
- U3: value MOC3023 -> MOC3163-M; Farnell 2322550 -> 1467853
- renumbered C2 to C1, C3 to C2, C4 to C3, C1 to C4, P3 to P1, P1 to P2, P2 to P3, R3 to R2, R7 to R3, R8 to R4, R9 to R5, R10 to R6, U5 to U2
Connections:
- net labels added: TEMP_SENSE
- net labels removed: XOVER_SENSE
- wire segments 124 -> 115
Other:
- note added: "1000V/us min critical rise\n5mA trigger current\n12V typical inhibit voltage\nDIP-6"
- note added: "In theory we only need 20mA\nhere, ignoring inrush or switching"
- note added: "POWER SUPPLY"
- note removed: "+6VAC (RMS)"
- note removed: "2.5VDC"
- note removed: "2.5VDC +\n1.4VAC_RMS"
- note removed: "POWER SUPPLY & CROSSOVER SENSE"
- note removed: "TODO: pick a decent opamp/comparator"

Commit message: Power footprints and associations
Also first thoughts on PCB shape and connector placement
Parts:
- removed P2: MAINS, symbol CONN_01X02
- removed P3: LOAD, symbol CONN_01X02
- added P2: MAINS_INLET, symbol CONN_01X03
- added P3: LOAD_OUTLET, symbol CONN_01X03
Connections:
- net labels added: EARTH
- wire segments 115 -> 119
Changed lines of the file:
@@
 $EndComp
-$Comp
-L CONN_01X02 P2
-U 1 1 54E56544
-P 1100 6550
-F 0 "P2" H 1100 6700 50  0000 C CNN
-F 1 "MAINS" V 1200 6550 50  0000 C CNN
-F 2 "" H 1100 6550 60  0000 C CNN
-F 3 "" H 1100 6550 60  0000 C CNN
-	1    1100 6550
-	-1   0    0    1
-$EndComp
-Text GLabel 2300 6450 2    60   Input ~ 0
-MAINS_LIVE
-Text GLabel 2300 6650 2    60   Input ~ 0
-MAINS_NEUTRAL
-$Comp
-L CONN_01X02 P3
-U 1 1 54E5722D
-P 4900 7100
-F 0 "P3" H 4900 7250 50  0000 C CNN
-F 1 "LOAD" V 5000 7100 50  0000 C CNN
-F 2 "" H 4900 7100 60  0000 C CNN
-F 3 "" H 4900 7100 60  0000 C CNN
-	1    4900 7100
-	1    0    0    -1
-$EndComp
-Text GLabel 4600 7200 0    60   Input ~ 0
-LOAD_LIVE
-Text GLabel 4600 7000 0    60   Input ~ 0
-LOAD_NEUTRAL
 $Comp
 L +5V #PWR02
 U 1 1 54E57BFD
-P 3700 6600
-F 0 "#PWR02" H 3700 6450 60  0001 C CNN
-F 1 "+5V" H 3700 6740 60  0000 C CNN
-F 2 "" H 3700 6600 60  0000 C CNN
-F 3 "" H 3700 6600 60  0000 C CNN
-	1    3700 6600
-	1    0    0    -1
-$EndComp
-Text GLabel 4700 6000 2    60   Input ~ 0
+P 1300 6450
+F 0 "#PWR02" H 1300 6300 60  0001 C CNN
+F 1 "+5V" H 1300 6590 60  0000 C CNN
+F 2 "" H 1300 6450 60  0000 C CNN
+F 3 "" H 1300 6450 60  0000 C CNN
+	1    1300 6450
+	1    0    0    -1
+$EndComp
+Text GLabel 2300 5850 2    60   Input ~ 0
 MASTER_RELAY
 $Comp
 L GND #PWR03
 U 1 1 54E58366
-P 3700 5850
-F 0 "#PWR03" H 3700 5600 60  0001 C CNN
-F 1 "GND" H 3700 5700 60  0000 C CNN
-F 2 "" H 3700 5850 60  0000 C CNN
-F 3 "" H 3700 5850 60  0000 C CNN
-	1    3700 5850
-	1    0    0    -1
-$EndComp
-Text GLabel 4700 6300 2    60   Input ~ 0
+P 1300 5700
+F 0 "#PWR03" H 1300 5450 60  0001 C CNN
+F 1 "GND" H 1300 5550 60  0000 C CNN
+F 2 "" H 1300 5700 60  0000 C CNN
+F 3 "" H 1300 5700 60  0000 C CNN
+	1    1300 5700
+	1    0    0    -1
+$EndComp
+Text GLabel 2300 6150 2    60   Input ~ 0
 TRIAC_TRIG
 Text GLabel 8800 1800 0    60   Input ~ 0
@@
 Text GLabel 9600 4000 0    60   Input ~ 0
 TRIAC_MAINS
-Text GLabel 4000 6300 0    60   Input ~ 0
+Text GLabel 1600 6150 0    60   Input ~ 0
 I_SENSE
 Text Notes 8050 6450 0    157  ~ 0
@@
 Text Notes 2050 5350 0    157  ~ 0
 CURRENT SENSE
-Text Notes 2250 7700 0    157  ~ 0
+Text Notes 3550 5750 0    157  ~ 0
 CONNECTORS
 $Comp
 L PWR_FLAG #FLG012
 U 1 1 54E8D577
-P 1350 6450
-F 0 "#FLG012" H 1350 6545 30  0001 C CNN
-F 1 "PWR_FLAG" H 1350 6630 30  0000 C CNN
-F 2 "" H 1350 6450 60  0000 C CNN
-F 3 "" H 1350 6450 60  0000 C CNN
-	1    1350 6450
+P 1650 6950
+F 0 "#FLG012" H 1650 7045 30  0001 C CNN
+F 1 "PWR_FLAG" H 1650 7130 30  0000 C CNN
+F 2 "" H 1650 6950 60  0000 C CNN
+F 3 "" H 1650 6950 60  0000 C CNN
+	1    1650 6950
 	1    0    0    -1
 $EndComp
@@
 L PWR_FLAG #FLG013
 U 1 1 54E8D5A7
-P 1350 6650
-F 0 "#FLG013" H 1350 6745 30  0001 C CNN
-F 1 "PWR_FLAG" H 1350 6830 30  0000 C CNN
-F 2 "" H 1350 6650 60  0000 C CNN
-F 3 "" H 1350 6650 60  0000 C CNN
-	1    1350 6650
-	-1   0    0    1
-$EndComp
-Text GLabel 4700 6150 2    60   Input ~ 0
+P 1900 6950
+F 0 "#FLG013" H 1900 7045 30  0001 C CNN
+F 1 "PWR_FLAG" H 1900 7130 30  0000 C CNN
+F 2 "" H 1900 6950 60  0000 C CNN
+F 3 "" H 1900 6950 60  0000 C CNN
+	1    1900 6950
+	1    0    0    -1
+$EndComp
+Text GLabel 2300 6000 2    60   Input ~ 0
 PREHEAT_RELAY
 Text GLabel 9000 3000 0    60   Input ~ 0
@@
 Text Notes 9500 2100 0    79   ~ 0
 MASTER NEUTRAL
-NoConn ~ 4600 6350
+NoConn ~ 2200 6200
 $Comp
 L BC817-40 Q2
@@
 L CONN_02X04 P1
 U 1 1 54E909DD
-P 4350 6200
-F 0 "P1" H 4350 6450 50  0000 C CNN
-F 1 "CONTROL" H 4350 5950 50  0000 C CNN
-F 2 "" H 4350 5000 60  0000 C CNN
-F 3 "" H 4350 5000 60  0000 C CNN
-	1    4350 6200
+P 1950 6050
+F 0 "P1" H 1950 6300 50  0000 C CNN
+F 1 "CONTROL" H 1950 5800 50  0000 C CNN
+F 2 "" H 1950 4850 60  0000 C CNN
+F 3 "" H 1950 4850 60  0000 C CNN
+	1    1950 6050
 	1    0    0    -1
 $EndComp
@@
 L FUSE F2
 U 1 1 54F25289
-P 1850 6450
-F 0 "F2" H 1950 6500 50  0000 C CNN
-F 1 "13A" H 1750 6400 50  0000 C CNN
-F 2 "" H 1850 6450 60  0000 C CNN
-F 3 "" H 1850 6450 60  0000 C CNN
-	1    1850 6450
+P 2150 7150
+F 0 "F2" H 2250 7200 50  0000 C CNN
+F 1 "13A" H 2050 7100 50  0000 C CNN
+F 2 "" H 2150 7150 60  0000 C CNN
+F 3 "" H 2150 7150 60  0000 C CNN
+	1    2150 7150
 	1    0    0    -1
 $EndComp
@@
 	7000 5050 7000 5100
 Wire Wire Line
-	1300 6500 1350 6500
-Wire Wire Line
-	1350 6500 1350 6450
-Wire Wire Line
-	1350 6450 1600 6450
-Wire Wire Line
-	1300 6600 1350 6600
-Wire Wire Line
-	1350 6600 1350 6650
-Wire Wire Line
-	1350 6650 2300 6650
-Wire Wire Line
-	4700 7150 4650 7150
-Wire Wire Line
-	4650 7150 4650 7200
-Wire Wire Line
-	4650 7200 4600 7200
-Wire Wire Line
-	4700 7050 4650 7050
-Wire Wire Line
-	4650 7050 4650 7000
-Wire Wire Line
-	4650 7000 4600 7000
-Wire Wire Line
 	8800 1800 9000 1800
 Wire Wire Line
@@
 	4750 3150 3550 3150
 Wire Wire Line
-	3950 5800 3950 6050
-Wire Wire Line
-	3950 5800 3700 5800
-Wire Wire Line
-	3700 5800 3700 5850
-Wire Wire Line
-	3950 6050 4100 6050
-Wire Wire Line
-	4100 6250 4050 6250
-Wire Wire Line
-	4050 6250 4050 6300
-Wire Wire Line
-	4050 6300 4000 6300
-Wire Wire Line
-	4600 6150 4700 6150
-Wire Wire Line
-	4600 6250 4650 6250
-Wire Wire Line
-	4650 6250 4650 6300
-Wire Wire Line
-	4650 6300 4700 6300
-Connection ~ 1350 6650
-Connection ~ 1350 6450
+	1550 5650 1550 5900
+Wire Wire Line
+	1550 5650 1300 5650
+Wire Wire Line
+	1300 5650 1300 5700
+Wire Wire Line
+	1550 5900 1700 5900
+Wire Wire Line
+	1700 6100 1650 6100
+Wire Wire Line
+	1650 6100 1650 6150
+Wire Wire Line
+	1650 6150 1600 6150
+Wire Wire Line
+	2200 6000 2300 6000
+Wire Wire Line
+	2200 6100 2250 6100
+Wire Wire Line
+	2250 6100 2250 6150
+Wire Wire Line
+	2250 6150 2300 6150
 Wire Wire Line
 	8650 4650 8650 4900
@@
 	10000 3100 10400 3100
 Wire Wire Line
-	4050 6350 4050 6600
-Wire Wire Line
-	4050 6350 4100 6350
+	1650 6200 1650 6450
+Wire Wire Line
+	1650 6200 1700 6200
 Wire Wire Line
 	8800 1050 9000 1050
@@
 Connection ~ 6800 1450
 Wire Wire Line
-	4600 6050 4650 6050
-Wire Wire Line
-	4650 6050 4650 6000
-Wire Wire Line
-	4650 6000 4700 6000
-Wire Wire Line
-	4050 6600 3700 6600
+	2200 5900 2250 5900
+Wire Wire Line
+	2250 5900 2250 5850
+Wire Wire Line
+	2250 5850 2300 5850
+Wire Wire Line
+	1650 6450 1300 6450
 Wire Notes Line
 	4200 3850 4200 4400
@@
 Wire Notes Line
 	5850 5450 500  5450
-Wire Wire Line
-	2100 6450 2300 6450
 Wire Wire Line
 	2150 1200 2350 1200
@@
 Wire Wire Line
 	9400 5850 9550 5850
-Text GLabel 4000 6150 0    60   Input ~ 0
+Text GLabel 1600 6000 0    60   Input ~ 0
 TEMP_SENSE
 Wire Wire Line
-	4000 6150 4100 6150
+	1600 6000 1700 6000
 Wire Wire Line
 	3250 1200 3250 1150
 Connection ~ 3250 1200
+$Comp
+L CONN_01X03 P2
+U 1 1 54F26236
+P 1500 7350
+F 0 "P2" H 1500 7550 50  0000 C CNN
+F 1 "MAINS_INLET" V 1600 7350 50  0000 C CNN
+F 2 "" H 1500 7350 60  0000 C CNN
+F 3 "" H 1500 7350 60  0000 C CNN
+F 4 "2080426" H 1500 7350 60  0001 C CNN "Farnell"
+	1    1500 7350
+	-1   0    0    1
+$EndComp
+$Comp
+L CONN_01X03 P3
+U 1 1 54F262A6
+P 4500 7350
+F 0 "P3" H 4500 7550 50  0000 C CNN
+F 1 "LOAD_OUTLET" V 4600 7350 50  0000 C CNN
+F 2 "" H 4500 7350 60  0000 C CNN
+F 3 "" H 4500 7350 60  0000 C CNN
+F 4 "2080465" H 4500 7350 60  0001 C CNN "Farnell"
+	1    4500 7350
+	1    0    0    1
+$EndComp
+Wire Wire Line
+	1700 7450 4300 7450
+Text Label 3200 7450 0    60   ~ 0
+EARTH
+Text GLabel 2450 7300 2    60   Input ~ 0
+MAINS_NEUTRAL
+Text GLabel 4150 7300 0    60   Input ~ 0
+LOAD_NEUTRAL
+Text GLabel 2450 7150 2    60   Input ~ 0
+MAINS_LIVE
+Text GLabel 3950 7150 0    60   Input ~ 0
+LOAD_LIVE
+Wire Wire Line
+	2400 7150 2450 7150
+Wire Wire Line
+	1700 7350 1950 7350
+Wire Wire Line
+	1950 7350 1950 7300
+Wire Wire Line
+	1950 7300 2450 7300
+Wire Wire Line
+	1900 7150 1900 7250
+Wire Wire Line
+	1900 7250 1700 7250
+Wire Wire Line
+	1650 6950 1750 6950
+Wire Wire Line
+	1750 6950 1750 7250
+Connection ~ 1750 7250
+Wire Wire Line
+	1900 6950 1850 6950
+Wire Wire Line
+	1850 6950 1850 7350
+Connection ~ 1850 7350
+Wire Wire Line
+	4150 7300 4200 7300
+Wire Wire Line
+	4200 7300 4200 7350
+Wire Wire Line
+	4200 7350 4300 7350
+Wire Wire Line
+	3950 7150 4250 7150
+Wire Wire Line
+	4250 7150 4250 7250
+Wire Wire Line
+	4250 7250 4300 7250
 $EndSCHEMATC
