File: power/power.sch (KiCad schematic (older format))
At the start: 26 parts, among them K1 RELAY_SPST, K2 RELAY_SPST, K3 RELAY_SPST, P1 CONTROL, P2 MAINS_INLET, P3 LOAD_OUTLET, Q1 BC817-40, Q2 BC817-40, Q3 BC817-40, U1 VTX214, U2 ACS710, U3 MOC3163-M, U4 TIC206M, U5 DS18B20

Commit message: Power: onboard fuses, better attempt at first pcb
Parts:
- F1: Farnell (none) -> 1162740
- F2: Farnell (none) -> 1603990
- K1: value RELAY_SPST -> MASTER_LIVE
- K2: value RELAY_SPST -> MASTER_NEUTRAL
- K3: value RELAY_SPST -> PREHEAT
Other:
- note removed: "In theory we only need 20mA\nhere, ignoring inrush or switching"
- note removed: "MASTER LIVE"
- note removed: "MASTER NEUTRAL"
- note removed: "PREHEAT"
Changed lines of the file:
@@
 	1    0    0    -1
 $EndComp
-Text Notes 9700 3300 0    79   ~ 0
-PREHEAT
-Text Notes 9500 2100 0    79   ~ 0
-MASTER NEUTRAL
 NoConn ~ 2200 6200
 $Comp
@@
 P 9600 3200
 F 0 "K3" H 9600 3500 50  0000 C CNN
-F 1 "RELAY_SPST" H 9750 2950 50  0000 C CNN
+F 1 "PREHEAT" H 9750 2950 50  0000 C CNN
 F 2 "" H 9600 3450 60  0000 C CNN
 F 3 "" H 9600 3450 60  0000 C CNN
@@
 	1    0    0    -1
 $EndComp
-Text Notes 9500 1350 0    79   ~ 0
-MASTER LIVE
 $Comp
 L BC817-40 Q1
@@
 P 9400 1250
 F 0 "K1" H 9400 1550 50  0000 C CNN
-F 1 "RELAY_SPST" H 9550 1000 50  0000 C CNN
+F 1 "MASTER_LIVE" H 9550 1000 50  0000 C CNN
 F 2 "" H 9400 1500 60  0000 C CNN
 F 3 "" H 9400 1500 60  0000 C CNN
@@
 P 9400 2000
 F 0 "K2" H 9400 2300 50  0000 C CNN
-F 1 "RELAY_SPST" H 9550 1750 50  0000 C CNN
+F 1 "MASTER_NEUTRAL" H 9550 1750 50  0000 C CNN
 F 2 "" H 9400 2250 60  0000 C CNN
 F 3 "" H 9400 2250 60  0000 C CNN
@@
 F 2 "" H 2150 7150 60  0000 C CNN
 F 3 "" H 2150 7150 60  0000 C CNN
+F 4 "1603990" H 2150 7150 60  0001 C CNN "Farnell"
 	1    2150 7150
 	1    0    0    -1
@@
 F 2 "" H 2600 1200 60  0000 C CNN
 F 3 "" H 2600 1200 60  0000 C CNN
+F 4 "1162740" H 2600 1200 60  0001 C CNN "Farnell"
 	1    2600 1200
 	1    0    0    -1
 $EndComp
-Text Notes 1600 850  0    60   ~ 0
-In theory we only need 20mA\nhere, ignoring inrush or switching
 $Comp
 L DS18B20 U5
@@
 	2150 1350 3100 1350
 Wire Notes Line
-	2250 900  2250 1300
-Wire Notes Line
-	2250 1300 2900 1300
-Wire Notes Line
-	2900 1300 2900 1100
-Wire Notes Line
-	2900 1100 2250 1100
-Wire Notes Line
 	9500 4850 9500 4950
