File: power/power.sch (KiCad schematic (older format))
At the start: 26 parts, among them K1 MASTER_LIVE, K2 MASTER_NEUTRAL, K3 PREHEAT, P1 CONTROL, P2 MAINS_INLET, P3 LOAD_OUTLET, Q1 BC817-40, Q2 BC817-40, Q3 BC817-40, U1 VTX214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

Commit message: Removed neutral switching, more pcb mains rev
Parts:
- removed K2: MASTER_NEUTRAL, symbol RELAY_SPST
- removed Q2: BC817-40, SOT-23, symbol BC817-40
- removed R2: 390R, symbol R
- C1, C2, C3: footprint (none) -> Capacitors_SMD:C_0805
- C4: footprint (none) -> Capacitors_SMD:C_1210
- F1: footprint (none) -> power:5x20_clip
- F2: footprint (none) -> power:BS1362_clip
- K1: footprint (none) -> power:RZ03-1A4
- K2: renamed from K3; footprint (none) -> power:RZ03-1A4
- P1: footprint (none) -> power:TS821X08XXS100
- P2: footprint (none) -> power:GSP1_9103
- P3: footprint (none) -> power:5001
- Q1: footprint SOT-23 -> power:SOT23
- Q2: renamed from Q3; footprint SOT-23 -> power:SOT23
- R1: footprint (none) -> Resistors_SMD:R_0805
- R2: renamed from R3; footprint (none) -> Resistors_SMD:R_0805
- R3: renamed from R4; footprint (none) -> Resistors_SMD:R_0805
- R4: renamed from R5; footprint (none) -> Capacitors_SMD:C_1206
- R5: renamed from R6; footprint (none) -> Capacitors_SMD:C_0805
- U1: footprint (none) -> power:VTX214
- U2: footprint (none) -> power:SOIC16W-chunky
- U3: footprint (none) -> Sockets_DIP:DIP-6__300_ELL
- U4: footprint (none) -> Transistors_TO-220:TO-220_Neutral123_Vertical_LargePads
- U5: footprint (none) -> power:to92-straight
Connections:
- net labels removed: SENSE_NEUTRAL
- wire segments 119 -> 110

Commit message: Power: Thermal switch based cutoff
Parts:
- removed U5: DS18B20, power:to92-straight, symbol DS18B20
- added U5: 70°C, Wire_Connections_Bridges:WireConnection_1mmDrill, symbol thermal_switch
- P1: Farnell (none) -> 2215303
Connections:
- net labels removed: TEMP_SENSE
- wire segments 110 -> 104
- no-connect marks 3 -> 4
Changed lines of the file:
@@
 LIBS:relay_spst
 LIBS:vtx214
-LIBS:ds18b20
+LIBS:thermal_switch
 LIBS:power-cache
 EELAYER 25 0
@@
 L TRIAC U4
 U 1 1 54E5283F
-P 9700 4700
-F 0 "U4" H 9450 5050 50  0000 C CNN
-F 1 "TIC206M" H 9900 4950 50  0000 C CNN
-F 2 "Transistors_TO-220:TO-220_Neutral123_Vertical_LargePads" H 9700 4700 60  0001 C CNN
-F 3 "" H 9700 4700 60  0000 C CNN
-	1    9700 4700
+P 9900 4700
+F 0 "U4" H 9650 5050 50  0000 C CNN
+F 1 "TIC206M" H 10100 4950 50  0000 C CNN
+F 2 "Transistors_TO-220:TO-220_Neutral123_Vertical_LargePads" H 9900 4700 60  0001 C CNN
+F 3 "" H 9900 4700 60  0000 C CNN
+	1    9900 4700
 	1    0    0    -1
 $EndComp
@@
 L OPTO-TRIAC U3
 U 1 1 54E528C7
-P 7850 4450
-F 0 "U3" H 8050 4750 60  0000 C CNN
-F 1 "MOC3163-M" H 7650 4750 60  0000 C CNN
-F 2 "Sockets_DIP:DIP-6__300_ELL" H 7850 4450 60  0001 C CNN
-F 3 "" H 7850 4450 60  0000 C CNN
-F 4 "1467853" H 7850 4450 60  0001 C CNN "Farnell"
-	1    7850 4450
+P 7350 4450
+F 0 "U3" H 7550 4750 60  0000 C CNN
+F 1 "MOC3163-M" H 7150 4750 60  0000 C CNN
+F 2 "Sockets_DIP:DIP-6__300_ELL" H 7350 4450 60  0001 C CNN
+F 3 "" H 7350 4450 60  0000 C CNN
+F 4 "1467853" H 7350 4450 60  0001 C CNN "Farnell"
+	1    7350 4450
 	1    0    0    -1
 $EndComp
@@
 L R R3
 U 1 1 54E52E94
-P 8900 4250
-F 0 "R3" V 8980 4250 50  0000 C CNN
-F 1 "390R" V 8800 4250 50  0000 C CNN
-F 2 "Resistors_SMD:R_0805" V 8830 4250 30  0001 C CNN
-F 3 "" H 8900 4250 30  0000 C CNN
-F 4 "2331790" H 8900 4250 60  0001 C CNN "Farnell"
-	1    8900 4250
+P 8250 4250
+F 0 "R3" V 8330 4250 50  0000 C CNN
+F 1 "390R" V 8150 4250 50  0000 C CNN
+F 2 "Resistors_SMD:R_0805" V 8180 4250 30  0001 C CNN
+F 3 "" H 8250 4250 30  0000 C CNN
+F 4 "2331790" H 8250 4250 60  0001 C CNN "Farnell"
+	1    8250 4250
 	0    1    1    0
 $EndComp
@@
 L R R4
 U 1 1 54E5366C
-P 10300 4750
-F 0 "R4" V 10380 4750 50  0000 C CNN
-F 1 "47R" V 10307 4751 50  0000 C CNN
-F 2 "Capacitors_SMD:C_1206" V 10230 4750 30  0001 C CNN
-F 3 "" H 10300 4750 30  0000 C CNN
-F 4 "1887414" H 10300 4750 60  0001 C CNN "Farnell"
-	1    10300 4750
+P 10500 4750
+F 0 "R4" V 10580 4750 50  0000 C CNN
+F 1 "47R" V 10507 4751 50  0000 C CNN
+F 2 "Capacitors_SMD:C_1206" V 10430 4750 30  0001 C CNN
+F 3 "" H 10500 4750 30  0000 C CNN
+F 4 "1887414" H 10500 4750 60  0001 C CNN "Farnell"
+	1    10500 4750
 	1    0    0    -1
 $EndComp
@@
 L C C4
 U 1 1 54E536C9
-P 10300 4250
-F 0 "C4" H 10350 4350 50  0000 L CNN
-F 1 "22nF" H 10350 4150 50  0000 L CNN
-F 2 "Capacitors_SMD:C_1210" H 10338 4100 30  0001 C CNN
-F 3 "" H 10300 4250 60  0000 C CNN
-F 4 "2057310" H 10300 4250 60  0001 C CNN "Farnell"
-	1    10300 4250
-	1    0    0    -1
-$EndComp
-Text GLabel 10350 5250 2    60   Input ~ 0
+P 10500 4250
+F 0 "C4" H 10550 4350 50  0000 L CNN
+F 1 "22nF" H 10550 4150 50  0000 L CNN
+F 2 "Capacitors_SMD:C_1210" H 10538 4100 30  0001 C CNN
+F 3 "" H 10500 4250 60  0000 C CNN
+F 4 "2057310" H 10500 4250 60  0001 C CNN "Farnell"
+	1    10500 4250
+	1    0    0    -1
+$EndComp
+Text GLabel 10550 5250 2    60   Input ~ 0
 LOAD_LIVE
-Text GLabel 7000 4250 0    60   Input ~ 0
+Text GLabel 6500 4250 0    60   Input ~ 0
 TRIAC_TRIG
 $Comp
 L R R5
 U 1 1 54E53E1C
-P 7000 4800
-F 0 "R5" V 7080 4800 50  0000 C CNN
-F 1 "220R" V 6900 4800 50  0000 C CNN
-F 2 "Capacitors_SMD:C_0805" V 6930 4800 30  0001 C CNN
-F 3 "" H 7000 4800 30  0000 C CNN
-F 4 "2331787" H 7000 4800 60  0001 C CNN "Farnell"
-	1    7000 4800
+P 6500 4800
+F 0 "R5" V 6580 4800 50  0000 C CNN
+F 1 "220R" V 6400 4800 50  0000 C CNN
+F 2 "Capacitors_SMD:C_0805" V 6430 4800 30  0001 C CNN
+F 3 "" H 6500 4800 30  0000 C CNN
+F 4 "2331787" H 6500 4800 60  0001 C CNN "Farnell"
+	1    6500 4800
 	1    0    0    -1
 $EndComp
@@
 L GND #PWR01
 U 1 1 54E54152
-P 7000 5100
-F 0 "#PWR01" H 7000 4850 60  0001 C CNN
-F 1 "GND" H 7000 4950 60  0000 C CNN
-F 2 "" H 7000 5100 60  0000 C CNN
-F 3 "" H 7000 5100 60  0000 C CNN
-	1    7000 5100
+P 6500 5100
+F 0 "#PWR01" H 6500 4850 60  0001 C CNN
+F 1 "GND" H 6500 4950 60  0000 C CNN
+F 2 "" H 6500 5100 60  0000 C CNN
+F 3 "" H 6500 5100 60  0000 C CNN
+	1    6500 5100
 	1    0    0    -1
 $EndComp
@@
 Text GLabel 10150 1550 2    60   Input ~ 0
 TRIAC_MAINS
-Text GLabel 9600 4000 0    60   Input ~ 0
+Text GLabel 9800 3900 0    60   Input ~ 0
 TRIAC_MAINS
 Text GLabel 1600 6150 0    60   Input ~ 0
@@
 F 2 "power:TS821X08XXS100" H 1950 4850 60  0001 C CNN
 F 3 "" H 1950 4850 60  0000 C CNN
+F 4 "2215303" H 1950 6050 60  0001 C CNN "Farnell"
 	1    1950 6050
 	1    0    0    -1
@@
 	1    0    0    -1
 $EndComp
-$Comp
-L DS18B20 U5
-U 1 1 54F27DA1
-P 9400 5100
-F 0 "U5" H 9400 5050 60  0000 C CNN
-F 1 "DS18B20" H 9400 5150 60  0000 C CNN
-F 2 "power:to92-straight" H 9400 5100 60  0001 C CNN
-F 3 "" H 9400 5100 60  0000 C CNN
-	1    9400 5100
-	1    0    0    -1
-$EndComp
-Wire Wire Line
-	8450 4250 8650 4250
-Wire Wire Line
-	8450 4650 8650 4650
-Wire Wire Line
-	10300 4450 10300 4500
-Wire Wire Line
-	9700 5050 10300 5050
-Wire Wire Line
-	10300 5050 10300 5000
-Wire Wire Line
-	9700 5250 10350 5250
-Connection ~ 9700 5050
-Wire Wire Line
-	7000 4250 7200 4250
-Wire Wire Line
-	7200 4550 7000 4550
-Wire Wire Line
-	7000 5050 7000 5100
+Wire Wire Line
+	7950 4250 8000 4250
+Wire Wire Line
+	7950 4650 8150 4650
+Wire Wire Line
+	10500 4450 10500 4500
+Wire Wire Line
+	9900 5050 10500 5050
+Wire Wire Line
+	10500 5050 10500 5000
+Wire Wire Line
+	9900 5250 10550 5250
+Connection ~ 9900 5050
+Wire Wire Line
+	6500 4250 6700 4250
+Wire Wire Line
+	6700 4550 6500 4550
+Wire Wire Line
+	6500 5050 6500 5100
 Wire Wire Line
 	2050 3100 1950 3100
@@
 	2250 6150 2300 6150
 Wire Wire Line
-	8650 4650 8650 4900
-Wire Wire Line
-	9700 4950 9700 5250
-Wire Wire Line
-	9600 4000 10300 4000
-Wire Wire Line
-	9700 4000 9700 4300
-Wire Wire Line
-	8650 4900 9200 4900
-Wire Wire Line
-	9150 4250 9700 4250
-Connection ~ 9700 4250
-Wire Wire Line
-	10300 4000 10300 4050
-Connection ~ 9700 4000
+	8150 4650 8150 4900
+Wire Wire Line
+	9900 4950 9900 5250
+Wire Wire Line
+	8150 4900 9400 4900
+Connection ~ 9900 4250
+Wire Wire Line
+	10500 3900 10500 4050
 Wire Wire Line
 	8850 2650 9050 2650
@@
 Wire Wire Line
 	2150 1350 3100 1350
-Wire Notes Line
-	9500 4850 9500 4950
-Wire Notes Line
-	9550 4800 9550 4950
-Wire Notes Line
-	9600 4800 9600 4950
-Wire Notes Line
-	9450 4900 9450 4950
-Text Notes 7250 5100 0    60   ~ 0
+Text Notes 6750 5100 0    60   ~ 0
 1000V/us min critical rise\n5mA trigger current\n12V typical inhibit voltage\nDIP-6
-$Comp
-L GND #PWR019
-U 1 1 54F2A019
-P 9250 5650
-F 0 "#PWR019" H 9250 5400 60  0001 C CNN
-F 1 "GND" H 9250 5500 60  0000 C CNN
-F 2 "" H 9250 5650 60  0000 C CNN
-F 3 "" H 9250 5650 60  0000 C CNN
-	1    9250 5650
-	1    0    0    -1
-$EndComp
-Wire Wire Line
-	9250 5600 9250 5650
-$Comp
-L +5V #PWR020
-U 1 1 54F2A0EF
-P 9750 5650
-F 0 "#PWR020" H 9750 5500 60  0001 C CNN
-F 1 "+5V" H 9750 5790 60  0000 C CNN
-F 2 "" H 9750 5650 60  0000 C CNN
-F 3 "" H 9750 5650 60  0000 C CNN
-	1    9750 5650
-	1    0    0    -1
-$EndComp
-Wire Wire Line
-	9550 5600 9550 5700
-Wire Wire Line
-	9550 5700 9750 5700
-Wire Wire Line
-	9750 5700 9750 5650
-Wire Wire Line
-	9400 5600 9400 5850
-Text GLabel 9550 5850 2    60   Input ~ 0
-TEMP_SENSE
-Wire Wire Line
-	9400 5850 9550 5850
-Text GLabel 1600 6000 0    60   Input ~ 0
-TEMP_SENSE
-Wire Wire Line
-	1600 6000 1700 6000
 Wire Wire Line
 	3250 1200 3250 1150
@@
 	1950 7300 2450 7300
 Wire Wire Line
-	1900 7150 1900 7250
-Wire Wire Line
-	1900 7250 1700 7250
+	1900 7250 1900 7150
+Wire Wire Line
+	1700 7250 1900 7250
 Wire Wire Line
 	1650 6950 1750 6950
@@
 Wire Wire Line
 	4250 7250 4300 7250
+$Comp
+L thermal_switch U5
+U 1 1 54F50713
+P 9000 4250
+F 0 "U5" H 8850 4400 60  0000 C CNN
+F 1 "70°C" H 9050 3950 60  0000 C CNN
+F 2 "Wire_Connections_Bridges:WireConnection_1mmDrill" H 8950 4800 60  0001 C CNN
+F 3 "" H 8950 4800 60  0000 C CNN
+F 4 "SN36219" H 9000 4250 60  0001 C CNN "Farnell"
+	1    9000 4250
+	1    0    0    -1
+$EndComp
+Wire Wire Line
+	9500 4250 9900 4250
+Wire Wire Line
+	9800 3900 10500 3900
+Wire Wire Line
+	9900 3900 9900 4300
+Wire Wire Line
+	8550 4250 8500 4250
+NoConn ~ 1700 6000
+Connection ~ 9900 3900
 $EndSCHEMATC

Commit message: Updated TRIAC part, added LEDs.
Parts:
- added D1: POWER, power:LED-0805, symbol LED
- added D2: MASTER, power:LED-0805, symbol LED
- added D3: PREHEAT, power:LED-0805, symbol LED
- added D4: TRIAC, power:LED-0805, symbol LED
- added R2, R3, R5: 300R, Resistors_SMD:R_0805, symbol R
- added R7: 75R, Resistors_SMD:R_0805, symbol R
- U5: renamed from U4; value TIC206M -> BTA16-800BRG; Farnell (none) -> 1057281
- renumbered R2 to R4, R3 to R6, R4 to R8, R5 to R9, U5 to U3, U3 to U4
Connections:
- wire segments 104 -> 118
Other:
- note added: "GREEN"
- note added: "ORANGE"
- note added: "RED"
- note added: "YELLOW"

Commit message: P: Updated connector footprint and pinout
Also decided to stick with ACS712 instead of cheaper/smaller ACS710 because the
former is SOICW instead of SOIC so has a bit more isolation distance.
Parts:
- P1: footprint power:TS821X08XXS100 -> control:2x4_100
Connections:
- wire segments 118 -> 115
Changed lines of the file:
@@
 L +5V #PWR18
 U 1 1 54E57BFD
-P 1300 6450
-F 0 "#PWR18" H 1300 6300 60  0001 C CNN
-F 1 "+5V" H 1300 6590 60  0000 C CNN
-F 2 "" H 1300 6450 60  0000 C CNN
-F 3 "" H 1300 6450 60  0000 C CNN
-	1    1300 6450
+P 2450 6450
+F 0 "#PWR18" H 2450 6300 60  0001 C CNN
+F 1 "+5V" H 2450 6590 60  0000 C CNN
+F 2 "" H 2450 6450 60  0000 C CNN
+F 3 "" H 2450 6450 60  0000 C CNN
+	1    2450 6450
 	1    0    0    -1
 $EndComp
@@
 Text GLabel 10100 4250 0    60   Input ~ 0
 TRIAC_MAINS
-Text GLabel 1600 6150 0    60   Input ~ 0
+Text GLabel 1600 6000 0    60   Input ~ 0
 I_SENSE
 Text Notes 8050 6450 0    157  ~ 0
@@
 	1    0    0    -1
 $EndComp
-NoConn ~ 2200 6200
 $Comp
 L BC817-40 Q2
@@
 F 0 "P1" H 1950 6300 50  0000 C CNN
 F 1 "CONTROL" H 1950 5800 50  0000 C CNN
-F 2 "power:TS821X08XXS100" H 1950 4850 60  0001 C CNN
+F 2 "control:2x4_100" H 1950 4850 60  0001 C CNN
 F 3 "" H 1950 4850 60  0000 C CNN
 F 4 "2215303" H 1950 6050 60  0001 C CNN "Farnell"
@@
 	1550 5900 1700 5900
 Wire Wire Line
-	1700 6100 1650 6100
-Wire Wire Line
-	1650 6100 1650 6150
-Wire Wire Line
-	1650 6150 1600 6150
-Wire Wire Line
 	2200 6000 2300 6000
 Wire Wire Line
@@
 	9900 2900 10300 2900
 Wire Wire Line
-	1650 6200 1650 6450
-Wire Wire Line
-	1650 6200 1700 6200
-Wire Wire Line
 	8750 1150 8950 1150
 Wire Wire Line
@@
 Wire Wire Line
 	2250 5850 2300 5850
-Wire Wire Line
-	1650 6450 1300 6450
 Wire Notes Line
 	4200 3850 4200 4400
@@
 Wire Wire Line
 	9050 4600 9000 4600
-NoConn ~ 1700 6000
 Connection ~ 10200 4250
 $Comp
@@
 Wire Wire Line
 	8450 3550 8450 3600
+Wire Wire Line
+	2200 6200 2200 6450
+Wire Wire Line
+	2200 6450 2450 6450
+NoConn ~ 1700 6200
+Wire Wire Line
+	1600 6000 1700 6000
+NoConn ~ 1700 6100
 $EndSCHEMATC

Commit message: Added *correct* heatsink to schematic.
Other:
- note added: "Heatsink:\n1703170"
Changed lines of the file:
@@
 	1600 6000 1700 6000
 NoConn ~ 1700 6100
+Text Notes 9650 5500 0    60   ~ 0
+Heatsink:\n1703170
 $EndSCHEMATC

Commit message: Mostly LED value fixes, relay transistors
Parts:
- R2, R3, R5: Farnell (none) -> 2138881
- R7: value 75R -> 300R; Farnell (none) -> 2138881
- R9: value 220R -> 300R
Connections:
- net labels removed: V_OFFSET
- wire segments 115 -> 118
Other:
- note added: "INSULATED TAB"

Commit message: Lots of footprint modifications
Parts:
- P2: footprint power:GSP1_9103 -> power:GSP1_9103_no_protrude
- P3: footprint power:5001 -> power:5001_no_protrude
Other:
- note added: "ISOLATED TAB"
- note removed: "INSULATED TAB"
Changed lines of the file:
@@
 F 0 "P2" H 1500 7550 50  0000 C CNN
 F 1 "MAINS_INLET" V 1600 7350 50  0000 C CNN
-F 2 "power:GSP1_9103" H 1500 7350 60  0001 C CNN
+F 2 "power:GSP1_9103_no_protrude" H 1500 7350 60  0001 C CNN
 F 3 "" H 1500 7350 60  0000 C CNN
 F 4 "2080426" H 1500 7350 60  0001 C CNN "Farnell"
@@
 F 0 "P3" H 4500 7550 50  0000 C CNN
 F 1 "LOAD_OUTLET" V 4600 7350 50  0000 C CNN
-F 2 "power:5001" H 4500 7350 60  0001 C CNN
+F 2 "power:5001_no_protrude" H 4500 7350 60  0001 C CNN
 F 3 "" H 4500 7350 60  0000 C CNN
 F 4 "2080465" H 4500 7350 60  0001 C CNN "Farnell"
@@
 	3800 3550 3800 3600
 Text Notes 9450 5450 0    60   ~ 0
-INSULATED TAB
+ISOLATED TAB
 $EndSCHEMATC

Commit message: Test points, rerouted relay drivers.
Parts:
- added P4: +5V, Connect:1pin, symbol TST
- added P5: GND, Connect:1pin, symbol TST
- added P6: I_SENSE, Connect:1pin, symbol TST
Connections:
- wire segments 118 -> 121
Changed lines of the file:
@@
 $EndComp
 $Comp
-L GND #PWR01
+L GND #PWR15
 U 1 1 54E54152
 P 7100 5450
-F 0 "#PWR01" H 7100 5200 60  0001 C CNN
+F 0 "#PWR15" H 7100 5200 60  0001 C CNN
 F 1 "GND" H 7100 5300 60  0000 C CNN
 F 2 "" H 7100 5450 60  0000 C CNN
@@
 $EndComp
 $Comp
-L +5V #PWR02
+L +5V #PWR18
 U 1 1 54E57BFD
 P 2450 6450
-F 0 "#PWR02" H 2450 6300 60  0001 C CNN
+F 0 "#PWR18" H 2450 6300 60  0001 C CNN
 F 1 "+5V" H 2450 6590 60  0000 C CNN
 F 2 "" H 2450 6450 60  0000 C CNN
@@
 MASTER_RELAY
 $Comp
-L GND #PWR03
+L GND #PWR16
 U 1 1 54E58366
 P 1300 5700
-F 0 "#PWR03" H 1300 5450 60  0001 C CNN
+F 0 "#PWR16" H 1300 5450 60  0001 C CNN
 F 1 "GND" H 1300 5550 60  0000 C CNN
 F 2 "" H 1300 5700 60  0000 C CNN
@@
 NoConn ~ 3550 3250
 $Comp
-L +5V #PWR04
+L +5V #PWR9
 U 1 1 54E6A742
 P 4750 3100
-F 0 "#PWR04" H 4750 2950 60  0001 C CNN
+F 0 "#PWR9" H 4750 2950 60  0001 C CNN
 F 1 "+5V" H 4750 3240 60  0000 C CNN
 F 2 "" H 4750 3100 60  0000 C CNN
@@
 $EndComp
 $Comp
-L GND #PWR05
+L GND #PWR14
 U 1 1 54E6AA04
 P 4750 4050
-F 0 "#PWR05" H 4750 3800 60  0001 C CNN
+F 0 "#PWR14" H 4750 3800 60  0001 C CNN
 F 1 "GND" H 4750 3900 60  0000 C CNN
 F 2 "" H 4750 4050 60  0000 C CNN
@@
 $EndComp
 $Comp
-L GND #PWR06
+L GND #PWR6
 U 1 1 54E6AAC6
 P 3750 2950
-F 0 "#PWR06" H 3750 2700 60  0001 C CNN
+F 0 "#PWR6" H 3750 2700 60  0001 C CNN
 F 1 "GND" H 3750 2800 60  0000 C CNN
 F 2 "" H 3750 2950 60  0000 C CNN
@@
 	1    0    0    -1
 $EndComp
-Text GLabel 3700 3300 2    60   Input ~ 0
+Text GLabel 4250 3300 2    60   Input ~ 0
 I_SENSE
 $Comp
@@
 $EndComp
 $Comp
-L GND #PWR07
+L GND #PWR13
 U 1 1 54E6D672
 P 4500 4050
-F 0 "#PWR07" H 4500 3800 60  0001 C CNN
+F 0 "#PWR13" H 4500 3800 60  0001 C CNN
 F 1 "GND" H 4500 3900 60  0000 C CNN
 F 2 "" H 4500 4050 60  0000 C CNN
@@
 $EndComp
 $Comp
-L GND #PWR08
+L GND #PWR12
 U 1 1 54E6EA77
 P 3800 4050
-F 0 "#PWR08" H 3800 3800 60  0001 C CNN
+F 0 "#PWR12" H 3800 3800 60  0001 C CNN
 F 1 "GND" H 3800 3900 60  0000 C CNN
 F 2 "" H 3800 4050 60  0000 C CNN
@@
 $EndComp
 $Comp
-L GND #PWR09
+L GND #PWR11
 U 1 1 54E6EBEB
 P 3600 4050
-F 0 "#PWR09" H 3600 3800 60  0001 C CNN
+F 0 "#PWR11" H 3600 3800 60  0001 C CNN
 F 1 "GND" H 3600 3900 60  0000 C CNN
 F 2 "" H 3600 4050 60  0000 C CNN
@@
 CONNECTORS
 $Comp
-L PWR_FLAG #FLG010
+L PWR_FLAG #FLG2
 U 1 1 54E8D577
 P 1650 6950
-F 0 "#FLG010" H 1650 7045 30  0001 C CNN
+F 0 "#FLG2" H 1650 7045 30  0001 C CNN
 F 1 "PWR_FLAG" H 1650 7130 30  0000 C CNN
 F 2 "" H 1650 6950 60  0000 C CNN
@@
 $EndComp
 $Comp
-L PWR_FLAG #FLG011
+L PWR_FLAG #FLG3
 U 1 1 54E8D5A7
 P 1900 6950
-F 0 "#FLG011" H 1900 7045 30  0001 C CNN
+F 0 "#FLG3" H 1900 7045 30  0001 C CNN
 F 1 "PWR_FLAG" H 1900 7130 30  0000 C CNN
 F 2 "" H 1900 6950 60  0000 C CNN
@@
 PREHEAT_RELAY
 $Comp
-L +5V #PWR012
+L +5V #PWR8
 U 1 1 54E9E5A8
 P 7250 3050
-F 0 "#PWR012" H 7250 2900 60  0001 C CNN
+F 0 "#PWR8" H 7250 2900 60  0001 C CNN
 F 1 "+5V" H 7250 3190 60  0000 C CNN
 F 2 "" H 7250 3050 60  0000 C CNN
@@
 $EndComp
 $Comp
-L +5V #PWR013
+L +5V #PWR2
 U 1 1 54E81E7C
 P 8800 1350
-F 0 "#PWR013" H 8800 1200 60  0001 C CNN
+F 0 "#PWR2" H 8800 1200 60  0001 C CNN
 F 1 "+5V" H 8800 1490 60  0000 C CNN
 F 2 "" H 8800 1350 60  0000 C CNN
@@
 $EndComp
 $Comp
-L GND #PWR014
+L GND #PWR5
 U 1 1 54E81E8B
 P 8900 2000
-F 0 "#PWR014" H 8900 1750 60  0001 C CNN
+F 0 "#PWR5" H 8900 1750 60  0001 C CNN
 F 1 "GND" H 8900 1850 60  0000 C CNN
 F 2 "" H 8900 2000 60  0000 C CNN
@@
 MAINS_NEUTRAL
 $Comp
-L +5V #PWR015
+L +5V #PWR1
 U 1 1 54EA4FAC
 P 5300 800
-F 0 "#PWR015" H 5300 650 60  0001 C CNN
+F 0 "#PWR1" H 5300 650 60  0001 C CNN
 F 1 "+5V" H 5300 940 60  0000 C CNN
 F 2 "" H 5300 800 60  0000 C CNN
@@
 $EndComp
 $Comp
-L GND #PWR016
+L GND #PWR4
 U 1 1 54EA4FE1
 P 5300 2000
-F 0 "#PWR016" H 5300 1750 60  0001 C CNN
+F 0 "#PWR4" H 5300 1750 60  0001 C CNN
 F 1 "GND" H 5300 1850 60  0000 C CNN
 F 2 "" H 5300 2000 60  0000 C CNN
@@
 $EndComp
 $Comp
-L PWR_FLAG #FLG017
+L PWR_FLAG #FLG1
 U 1 1 54EA5407
 P 3250 1150
-F 0 "#FLG017" H 3250 1245 30  0001 C CNN
+F 0 "#FLG1" H 3250 1245 30  0001 C CNN
 F 1 "PWR_FLAG" H 3250 1330 30  0000 C CNN
 F 2 "" H 3250 1150 60  0000 C CNN
@@
 	3650 3350 3650 3300
 Wire Wire Line
-	3650 3300 3700 3300
+	3650 3300 4250 3300
 Wire Wire Line
 	4500 3450 4500 3600
@@
 	4900 1300 4900 1950
 Wire Wire Line
-	4900 1200 4500 1200
-Wire Wire Line
-	4900 850  4900 1200
+	4500 1200 4900 1200
+Wire Wire Line
+	4900 1200 4900 850
 Wire Notes Line
 	5850 7750 5850 500
@@
 $EndComp
 $Comp
-L GND #PWR018
+L GND #PWR17
 U 1 1 54F7A52B
 P 6600 5700
-F 0 "#PWR018" H 6600 5450 60  0001 C CNN
+F 0 "#PWR17" H 6600 5450 60  0001 C CNN
 F 1 "GND" H 6600 5550 60  0000 C CNN
 F 2 "" H 6600 5700 60  0000 C CNN
@@
 	8800 1350 8950 1350
 $Comp
-L +5V #PWR019
+L +5V #PWR3
 U 1 1 55175639
 P 7200 1450
-F 0 "#PWR019" H 7200 1300 60  0001 C CNN
+F 0 "#PWR3" H 7200 1300 60  0001 C CNN
 F 1 "+5V" H 7200 1590 60  0000 C CNN
 F 2 "" H 7200 1450 60  0000 C CNN
@@
 	7800 3100 7850 3100
 $Comp
-L +5V #PWR020
+L +5V #PWR7
 U 1 1 55176C80
 P 8950 3000
-F 0 "#PWR020" H 8950 2850 60  0001 C CNN
+F 0 "#PWR7" H 8950 2850 60  0001 C CNN
 F 1 "+5V" H 8950 3140 60  0000 C CNN
 F 2 "" H 8950 3000 60  0000 C CNN
@@
 	9100 2750 9100 2800
 $Comp
-L GND #PWR021
+L GND #PWR10
 U 1 1 551772AB
 P 9050 3650
-F 0 "#PWR021" H 9050 3400 60  0001 C CNN
+F 0 "#PWR10" H 9050 3400 60  0001 C CNN
 F 1 "GND" H 9050 3500 60  0000 C CNN
 F 2 "" H 9050 3650 60  0000 C CNN
@@
 Text Notes 9450 5450 0    60   ~ 0
 ISOLATED TAB
+$Comp
+L TST P4
+U 1 1 551891FA
+P 4650 1150
+F 0 "P4" H 4650 1450 50  0000 C BNN
+F 1 "+5V" H 4650 1400 50  0000 C CNN
+F 2 "Connect:1pin" H 4650 1150 60  0000 C CNN
+F 3 "" H 4650 1150 60  0000 C CNN
+	1    4650 1150
+	1    0    0    -1
+$EndComp
+$Comp
+L TST P5
+U 1 1 55189243
+P 4650 1350
+F 0 "P5" H 4650 1650 50  0000 C BNN
+F 1 "GND" H 4650 1600 50  0000 C CNN
+F 2 "Connect:1pin" H 4650 1350 60  0000 C CNN
+F 3 "" H 4650 1350 60  0000 C CNN
+	1    4650 1350
+	-1   0    0    1
+$EndComp
+Wire Wire Line
+	4650 1350 4650 1300
+Connection ~ 4650 1300
+Wire Wire Line
+	4650 1150 4650 1200
+Connection ~ 4650 1200
+$Comp
+L TST P6
+U 1 1 551895A8
+P 4100 3100
+F 0 "P6" H 4100 3400 50  0000 C BNN
+F 1 "I_SENSE" H 4100 3350 50  0000 C CNN
+F 2 "Connect:1pin" H 4100 3100 60  0000 C CNN
+F 3 "" H 4100 3100 60  0000 C CNN
+	1    4100 3100
+	1    0    0    -1
+$EndComp
+Wire Wire Line
+	4100 3100 4100 3300
+Connection ~ 4100 3300
 $EndSCHEMATC
