File: power/power.sch (KiCad schematic (older format))
At the start: 34 parts, among them K1 MASTER_LIVE, K2 PREHEAT, P1 CONTROL, P2 MAINS_INLET, P3 LOAD_OUTLET, P4 +5V, P5 GND, P6 I_SENSE, Q1 BC817-40, Q2 BC817-40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

Commit message: Power: Added relay flyback diodes.  Fixes #10
Parts:
- added D5, D6: MBR2H200SFT1G, power:SOD-123FL, symbol D_Schottky_Small
- C1, C2, C3, C4: symbol C -> C-RESCUE-power
- D1, D2, D3, D4: symbol LED -> LED-RESCUE-power
- R1, R2, R3, R4, R5, R6, R7, R8, R9: symbol R -> R-RESCUE-power
- U4: symbol OPTO-TRIAC -> OPTO-TRIAC-RESCUE-power
Connections:
- wire segments 121 -> 125
Changed lines of the file:
@@
 EESchema Schematic File Version 2
+LIBS:power-rescue
 LIBS:power
 LIBS:device
@@
 LIBS:memory
 LIBS:xilinx
-LIBS:special
 LIBS:microcontrollers
 LIBS:dsp
@@
 $EndComp
 $Comp
-L OPTO-TRIAC U4
+L OPTO-TRIAC-RESCUE-power U4
 U 1 1 54E528C7
 P 7850 4800
@@
 $EndComp
 $Comp
-L R R6
+L R-RESCUE-power R6
 U 1 1 54E52E94
 P 8750 4600
@@
 MAINS_LIVE
 $Comp
-L R R8
+L R-RESCUE-power R8
 U 1 1 54E5366C
 P 10800 5100
@@
 $EndComp
 $Comp
-L C C4
+L C-RESCUE-power C4
 U 1 1 54E536C9
 P 10800 4600
@@
 TRIAC_TRIG
 $Comp
-L R R9
+L R-RESCUE-power R9
 U 1 1 54E53E1C
 P 7100 5150
@@
 $EndComp
 $Comp
-L C C3
+L C-RESCUE-power C3
 U 1 1 54E6A771
 P 4750 3800
@@
 I_SENSE
 $Comp
-L C C2
+L C-RESCUE-power C2
 U 1 1 54E6D133
 P 4500 3800
@@
 $EndComp
 $Comp
-L C C1
+L C-RESCUE-power C1
 U 1 1 54E6E944
 P 3800 3800
@@
 $EndComp
 $Comp
-L R R4
+L R-RESCUE-power R4
 U 1 1 54E9E5AF
 P 8350 3400
@@
 $EndComp
 $Comp
-L R R1
+L R-RESCUE-power R1
 U 1 1 54E81E83
 P 8300 1750
@@
 Connection ~ 10200 4250
 $Comp
-L LED D1
+L LED-RESCUE-power D1
 U 1 1 54F7858E
 P 5300 1100
@@
 $EndComp
 $Comp
-L R R3
+L R-RESCUE-power R3
 U 1 1 54F785C7
 P 5300 1600
@@
 Connection ~ 5300 1950
 $Comp
-L R R2
+L R-RESCUE-power R2
 U 1 1 54F78EB6
 P 8100 1450
@@
 $EndComp
 $Comp
-L LED D2
+L LED-RESCUE-power D2
 U 1 1 54F78F0F
 P 7600 1450
@@
 $EndComp
 $Comp
-L R R5
+L R-RESCUE-power R5
 U 1 1 54F794DF
 P 8100 3100
@@
 $EndComp
 $Comp
-L LED D3
+L LED-RESCUE-power D3
 U 1 1 54F7952C
 P 7600 3100
@@
 	10200 5600 10400 5600
 $Comp
-L R R7
+L R-RESCUE-power R7
 U 1 1 54F7A4A8
 P 6600 4950
@@
 $EndComp
 $Comp
-L LED D4
+L LED-RESCUE-power D4
 U 1 1 54F7A4E7
 P 6600 5450
@@
 	8950 1100 8950 1150
 Wire Wire Line
-	8800 1350 8950 1350
+	8700 1350 8950 1350
 $Comp
 L +5V #PWR3
@@
 $EndComp
 Wire Wire Line
-	9100 3000 8950 3000
+	8900 3000 9100 3000
 Wire Wire Line
 	8900 2750 9100 2750
@@
 F 0 "P4" H 4650 1450 50  0000 C BNN
 F 1 "+5V" H 4650 1400 50  0000 C CNN
-F 2 "Connect:1pin" H 4650 1150 60  0000 C CNN
+F 2 "Connect:1pin" H 4650 1150 60  0001 C CNN
 F 3 "" H 4650 1150 60  0000 C CNN
 	1    4650 1150
@@
 F 0 "P5" H 4650 1650 50  0000 C BNN
 F 1 "GND" H 4650 1600 50  0000 C CNN
-F 2 "Connect:1pin" H 4650 1350 60  0000 C CNN
+F 2 "Connect:1pin" H 4650 1350 60  0001 C CNN
 F 3 "" H 4650 1350 60  0000 C CNN
 	1    4650 1350
@@
 F 0 "P6" H 4100 3400 50  0000 C BNN
 F 1 "I_SENSE" H 4100 3350 50  0000 C CNN
-F 2 "Connect:1pin" H 4100 3100 60  0000 C CNN
+F 2 "Connect:1pin" H 4100 3100 60  0001 C CNN
 F 3 "" H 4100 3100 60  0000 C CNN
 	1    4100 3100
@@
 	4100 3100 4100 3300
 Connection ~ 4100 3300
+$Comp
+L D_Schottky_Small D5
+U 1 1 55B7E4C8
+P 8625 1350
+F 0 "D5" H 8575 1250 50  0000 L CNN
+F 1 "MBR2H200SFT1G" H 8345 1270 50  0001 L CNN
+F 2 "power:SOD-123FL" V 8625 1350 60  0001 C CNN
+F 3 "" V 8625 1350 60  0000 C CNN
+F 4 "2452032" H 8625 1350 60  0001 C CNN "Farnell"
+	1    8625 1350
+	0    1    1    0
+$EndComp
+Connection ~ 8625 1450
+Wire Wire Line
+	8625 1250 8700 1250
+Wire Wire Line
+	8700 1250 8700 1350
+Connection ~ 8800 1350
+$Comp
+L D_Schottky_Small D6
+U 1 1 55B7F5FB
+P 8825 3000
+F 0 "D6" H 8775 2900 50  0000 L CNN
+F 1 "MBR2H200SFT1G" H 8545 2920 50  0001 L CNN
+F 2 "power:SOD-123FL" V 8825 3000 60  0001 C CNN
+F 3 "" V 8825 3000 60  0000 C CNN
+F 4 "2452032" H 8825 3000 60  0001 C CNN "Farnell"
+	1    8825 3000
+	0    1    1    0
+$EndComp
+Wire Wire Line
+	8825 2900 8900 2900
+Wire Wire Line
+	8900 2900 8900 3000
+Connection ~ 8950 3000
+Connection ~ 8825 3100
 $EndSCHEMATC

Commit message: Fixed R9 part number. Fixes #26
Parts:
- R9: Farnell 2331787 -> 2138881
Changed lines of the file:
@@
 F 2 "Capacitors_SMD:C_0805" V 7030 5150 30  0001 C CNN
 F 3 "" H 7100 5150 30  0000 C CNN
-F 4 "2331787" H 7100 5150 60  0001 C CNN "Farnell"
+F 4 "2138881" H 7100 5150 60  0001 C CNN "Farnell"
 	1    7100 5150
 	1    0    0    -1
