File: control/control.sch (KiCad schematic (older format))
At the start: 50 parts, among them CON1 USB-MICRO-B, IC1 STM32F072CBT6, IC2 AD8495, IC3 ADP3335, P1 SWD, P2 CONN_02X04, P3 CONN_01X02, Q1 NPN, U1 ROTENC, U2 ESP8266, U3 ER-OLED015-2B, X1 8MHz

Commit message: update sch: new oled, sync conditioning
Parts:
- removed C12, C19: 4µ7, symbol C
- removed C13, C21: 100n, symbol C
- removed C20: 10µ, symbol C
- removed R8: 910k, symbol R
- removed U3: ER-OLED015-2B, symbol ER-OLED015-2B
- added BT?: BATTERY, symbol BATTERY
- added C? (x2): 5p, symbol C
- added C? (x2): 100n, symbol C
- added R? (x3): 10k, symbol R
- added R?: 30k, symbol R
- added U?: ER-OLEDM024-2, symbol ER-OLEDM024-2
- added X?: 32k768, symbol CRYSTAL
- R2: value R -> 100
Connections:
- net labels added: OLED_E, ~OLED_CS, ~OLED_RST
- net labels removed: OLED_CS, OLED_E/RD, OLED_RES
- wire segments 229 -> 231
- no-connect marks 12 -> 10
Other:
- note added: "+5V from USB here so can be shorted to\nVCC for development, leave NC on power board"
- note added: "6800 Mode:\nBS1=0 BS2=1"
- note added: "Check SYNC, CURRENT, RELAY, TRIAC\nvoltage levels/specs"
- note removed: "+5V from USB here so can be shorted to\nVCC for development, leave NC on power"
- note removed: "Assumes 5V from power, but\nmaybe we need 12V for OLED"
- note removed: "Check PB[0:7] DMA"
- note removed: "Check SYNC OK\nwith COMP here"
- note removed: "Check SYNC, CURRENT, RELAY, TRIAC\nvoltage levels/specs\n(might need biasing on SYNC)"
- note removed: "Check TIM1_CH[1:3]N\nOK for PWM"
- note removed: "Check TIM3_CH[1:2] OK\nfor rotary encoder"
- note removed: "Consider 4wire SPI instead\n(might DMA better wrt clocks)\n\nThink about display interface,\n68xx or 80xx?"
- note removed: "IREF might want\nchanging for 5V VCC"
- note removed: "This is probably all OK"
- note removed: "add USB protection circuitry?"
- note removed: "no need for\nDP/DM resistors"
- note removed: "reconsider the 100n Cs"

Commit message: update sch: connection to power board
Parts:
- removed C?: 100n, symbol C
- removed R? (x3): 10k, symbol R
- removed R?: 30k, symbol R
Connections:
- wire segments 231 -> 224
Other:
- note removed: "Check SYNC, CURRENT, RELAY, TRIAC\nvoltage levels/specs"
- note removed: "Spec transistor driving"
Changed lines of the file:
@@
 L CONN_02X04 P2
 U 1 1 54D06BFB
-P 7150 4150
-F 0 "P2" H 7150 4400 50  0000 C CNN
-F 1 "CONN_02X04" H 7150 3900 50  0000 C CNN
-F 2 "" H 7150 2950 60  0000 C CNN
-F 3 "" H 7150 2950 60  0000 C CNN
-	1    7150 4150
+P 6500 4000
+F 0 "P2" H 6500 4250 50  0000 C CNN
+F 1 "CONN_02X04" H 6500 3750 50  0000 C CNN
+F 2 "" H 6500 2800 60  0000 C CNN
+F 3 "" H 6500 2800 60  0000 C CNN
+	1    6500 4000
 	1    0    0    -1
 $EndComp
@@
 L GND #PWR22
 U 1 1 54D0F836
-P 6550 4000
-F 0 "#PWR22" H 6550 3750 60  0001 C CNN
-F 1 "GND" H 6550 3850 60  0000 C CNN
-F 2 "" H 6550 4000 60  0000 C CNN
-F 3 "" H 6550 4000 60  0000 C CNN
-	1    6550 4000
+P 5900 3850
+F 0 "#PWR22" H 5900 3600 60  0001 C CNN
+F 1 "GND" H 5900 3700 60  0000 C CNN
+F 2 "" H 5900 3850 60  0000 C CNN
+F 3 "" H 5900 3850 60  0000 C CNN
+	1    5900 3850
 	0    1    1    0
 $EndComp
@@
 L VCC #PWR25
 U 1 1 54D0FA8C
-P 6800 4300
-F 0 "#PWR25" H 6800 4150 60  0001 C CNN
-F 1 "VCC" H 6800 4450 60  0000 C CNN
-F 2 "" H 6800 4300 60  0000 C CNN
-F 3 "" H 6800 4300 60  0000 C CNN
-	1    6800 4300
+P 6150 4150
+F 0 "#PWR25" H 6150 4000 60  0001 C CNN
+F 1 "VCC" H 6150 4300 60  0000 C CNN
+F 2 "" H 6150 4150 60  0000 C CNN
+F 3 "" H 6150 4150 60  0000 C CNN
+	1    6150 4150
 	0    -1   -1   0
 $EndComp
@@
 L +5V #PWR26
 U 1 1 54D0FED5
-P 7500 4300
-F 0 "#PWR26" H 7500 4150 60  0001 C CNN
-F 1 "+5V" H 7500 4440 60  0000 C CNN
-F 2 "" H 7500 4300 60  0000 C CNN
-F 3 "" H 7500 4300 60  0000 C CNN
-	1    7500 4300
+P 6850 4150
+F 0 "#PWR26" H 6850 4000 60  0001 C CNN
+F 1 "+5V" H 6850 4290 60  0000 C CNN
+F 2 "" H 6850 4150 60  0000 C CNN
+F 3 "" H 6850 4150 60  0000 C CNN
+	1    6850 4150
 	0    1    1    0
 $EndComp
-NoConn ~ 7400 4200
-Text Label 7550 4000 0    60   ~ 0
+NoConn ~ 6750 4050
+Text Label 6900 3850 0    60   ~ 0
 RELAY
-Text Label 7550 4100 0    60   ~ 0
+Text Label 6900 3950 0    60   ~ 0
 TRIAC
-Text Label 4850 4100 2    60   ~ 0
+Text Label 6100 3950 2    60   ~ 0
 SYNC
-Text Label 6750 4200 2    60   ~ 0
+Text Label 6100 4050 2    60   ~ 0
 CURRENT
 $Comp
@@
 NoConn ~ 8100 2850
 NoConn ~ 8100 2950
-Text Notes 6250 4650 0    60   ~ 0
+Text Notes 5600 4500 0    60   ~ 0
 +5V from USB here so can be shorted to\nVCC for development, leave NC on power board
-Text Notes 6350 3800 0    60   ~ 0
-Check SYNC, CURRENT, RELAY, TRIAC\nvoltage levels/specs
 $Comp
 L C C2
@@
 	1    0    0    -1
 $EndComp
-Text Notes 9150 1250 0    60   ~ 0
-Spec transistor driving
 Text Notes 550  5050 0    100  ~ 0
 MICROCONTROLLER
@@
 	4750 2450 4800 2450
 Wire Wire Line
-	6550 4000 6900 4000
-Wire Wire Line
-	6800 4300 6900 4300
+	5900 3850 6250 3850
+Wire Wire Line
+	6150 4150 6250 4150
 Wire Wire Line
 	7050 2500 7050 2550
@@
 	7050 2550 7100 2550
 Wire Wire Line
-	7400 4300 7500 4300
-Wire Wire Line
-	7400 4000 7550 4000
-Wire Wire Line
-	7400 4100 7550 4100
-Wire Wire Line
-	6000 4100 6900 4100
-Wire Wire Line
-	6900 4200 6750 4200
+	6750 4150 6850 4150
+Wire Wire Line
+	6750 3850 6900 3850
+Wire Wire Line
+	6750 3950 6900 3950
+Wire Wire Line
+	6250 4050 6100 4050
 Wire Wire Line
 	4800 1500 4850 1500
@@
 	1200 3850 1150 3850
 Connection ~ 1150 3850
-$Comp
-L C C?
-U 1 1 54DEC866
-P 5200 4100
-F 0 "C?" H 5250 4200 50  0000 L CNN
-F 1 "100n" H 5250 4000 50  0000 L CNN
-F 2 "" H 5238 3950 30  0000 C CNN
-F 3 "" H 5200 4100 60  0000 C CNN
-	1    5200 4100
-	0    1    1    0
-$EndComp
-$Comp
-L R R?
-U 1 1 54DEC901
-P 4950 3800
-F 0 "R?" V 5030 3800 50  0000 C CNN
-F 1 "10k" V 4957 3801 50  0000 C CNN
-F 2 "" V 4880 3800 30  0000 C CNN
-F 3 "" H 4950 3800 30  0000 C CNN
-	1    4950 3800
-	1    0    0    -1
-$EndComp
-$Comp
-L R R?
-U 1 1 54DEC9A4
-P 4950 4400
-F 0 "R?" V 5030 4400 50  0000 C CNN
-F 1 "10k" V 4957 4401 50  0000 C CNN
-F 2 "" V 4880 4400 30  0000 C CNN
-F 3 "" H 4950 4400 30  0000 C CNN
-	1    4950 4400
-	1    0    0    -1
-$EndComp
-$Comp
-L R R?
-U 1 1 54DEE5E1
-P 5750 4100
-F 0 "R?" V 5830 4100 50  0000 C CNN
-F 1 "30k" V 5757 4101 50  0000 C CNN
-F 2 "" V 5680 4100 30  0000 C CNN
-F 3 "" H 5750 4100 30  0000 C CNN
-	1    5750 4100
-	0    1    1    0
-$EndComp
-$Comp
-L R R?
-U 1 1 54DEE5E7
-P 5450 4400
-F 0 "R?" V 5530 4400 50  0000 C CNN
-F 1 "10k" V 5457 4401 50  0000 C CNN
-F 2 "" V 5380 4400 30  0000 C CNN
-F 3 "" H 5450 4400 30  0000 C CNN
-	1    5450 4400
-	1    0    0    -1
-$EndComp
-$Comp
-L VDD #PWR?
-U 1 1 54DEEEEF
-P 4950 3500
-F 0 "#PWR?" H 4950 3350 60  0001 C CNN
-F 1 "VDD" H 4950 3650 60  0000 C CNN
-F 2 "" H 4950 3500 60  0000 C CNN
-F 3 "" H 4950 3500 60  0000 C CNN
-	1    4950 3500
-	1    0    0    -1
-$EndComp
-$Comp
-L GND #PWR?
-U 1 1 54DEF184
-P 4950 4700
-F 0 "#PWR?" H 4950 4450 60  0001 C CNN
-F 1 "GND" H 4950 4550 60  0000 C CNN
-F 2 "" H 4950 4700 60  0000 C CNN
-F 3 "" H 4950 4700 60  0000 C CNN
-	1    4950 4700
-	1    0    0    -1
-$EndComp
-Wire Wire Line
-	4950 4650 4950 4700
-$Comp
-L GND #PWR?
-U 1 1 54DEF645
-P 5450 4700
-F 0 "#PWR?" H 5450 4450 60  0001 C CNN
-F 1 "GND" H 5450 4550 60  0000 C CNN
-F 2 "" H 5450 4700 60  0000 C CNN
-F 3 "" H 5450 4700 60  0000 C CNN
-	1    5450 4700
-	1    0    0    -1
-$EndComp
-Wire Wire Line
-	5450 4650 5450 4700
-Wire Wire Line
-	5400 4100 5500 4100
-Wire Wire Line
-	5450 4150 5450 4100
-Connection ~ 5450 4100
-Wire Wire Line
-	4850 4100 5000 4100
-Wire Wire Line
-	4950 4050 4950 4150
-Connection ~ 4950 4100
-Wire Wire Line
-	4950 3550 4950 3500
 $Comp
 L ER-OLEDM024-2 U?
@@
 Wire Wire Line
 	9650 2950 9650 3000
+Wire Wire Line
+	6100 3950 6250 3950
 $EndSCHEMATC

Commit message: further work on control, start routing pcb
Parts:
- removed U?: ER-OLEDM024-2, symbol ER-OLEDM024-2
- added C20: 100n, control:C0603, symbol C
- added U3: ER-OLEDM023-1, control:ER-OLEDM023-1, symbol ER-OLEDM023-1
- added U4: IDC SKT, symbol PART
- added U5, U6, U7, U8: M3_HOLE, control:M3_MOUNT, symbol PART
- BT1: renamed from BT?; footprint (none) -> control:2032HOLDER_KS1060; Farnell (none) -> 1704232
- C1, C14, C5, C6, C8, C9: footprint (none) -> control:C0603; Farnell (none) -> 1759122
- C10, C11: footprint (none) -> control:C0603; Farnell (none) -> 1759055
- C12, C13: renamed from C?; value 5p -> 15p; footprint (none) -> control:C0603; Farnell (none) -> 1759055
- C15, C26: footprint (none) -> control:C0603; Farnell (none) -> 2211164
- C16, C22: footprint (none) -> control:C1206; Farnell (none) -> 2211074
- C17, C18, C4: footprint (none) -> control:C0603; Farnell (none) -> 2346895
- C19: renamed from C?; footprint (none) -> control:C0603; Farnell (none) -> 1759122
- C2, C3: value 4µ7 -> 10µ; footprint (none) -> control:C0603; Farnell (none) -> 2211164
- C23, C25: footprint (none) -> control:C0603; Farnell (none) -> 2320817
- C24: footprint (none) -> control:C0603; Farnell (none) -> 1414605
- C7: footprint (none) -> control:C0603; Farnell (none) -> 2112704
- CON1: footprint (none) -> control:USB3065; Farnell (none) -> 2443120
- D1, D2: footprint (none) -> control:R0402; Farnell (none) -> 2368169
- IC1: footprint (none) -> control:LQFP48; Farnell (none) -> 2432094
- IC2: footprint (none) -> control:MSOP8; Farnell (none) -> 2067807
- IC3: footprint (none) -> control:MSOP8; Farnell (none) -> 2067775
- P1: footprint (none) -> control:FTSH-105-01-F-D-K; Farnell (none) -> 1667759
- P2: footprint (none) -> control:2x4_100; Farnell (none) -> 2215303
- P3: footprint (none) -> control:TC_K_PM; Farnell (none) -> 2347134
- Q1: footprint (none) -> control:SOT23; Farnell (none) -> 1081223
- R1, R3, R6: footprint (none) -> control:R0603; Farnell (none) -> 2332016
- R2, R4: footprint (none) -> control:R0603; Farnell (none) -> 2331989
- R5, R7: footprint (none) -> control:R0603; Farnell (none) -> 2116678
- R9: footprint (none) -> control:R0603; Farnell (none) -> 2321755
- SP1: footprint (none) -> control:ABT-402-RC; Farnell (none) -> 1022401
- U1: footprint (none) -> control:SF_ROTENC
- U2: footprint (none) -> control:ESP8266
- X1: footprint (none) -> control:XTAL50x32; Farnell (none) -> 2101329
- X2: renamed from X?; footprint (none) -> control:SMD_XTAL_8038; Farnell (none) -> 2308714
Connections:
- net labels added: M_RELAY, OLED_MOSI, OLED_SCLK, PH_RELAY
- net labels removed: OLED_D0, OLED_D1, OLED_D2, OLED_D3, OLED_D4, OLED_D5, OLED_D6, OLED_D7, OLED_E, OLED_R/W, RELAY
- no-connect marks 10 -> 15
Other:
- note added: "Set BS1=BS2=0 for SPI\n(solder jumpers on OLED PCB)"
- note removed: "6800 Mode:\nBS1=0 BS2=1"

Commit message: first routing complete!
Parts:
- removed Q1: NPN, control:SOT23, symbol NPN
- removed R2: 100, control:R0603, symbol R
- added IC1: AD8542, control:MSOP8, symbol AD8542
- added R1, R5: 15k, control:R0603, symbol R
- added R3, R6: 10k, control:R0603, symbol R
- renumbered C9 to C10, C12 to C11, C13 to C12, C19 to C13, C10 to C14, C11 to C15, C14 to C16, C15 to C17, C23 to C18, C24 to C19, C8 to C2, C25 to C20, C26 to C21, C16 to C22, C17 to C23, C18 to C24, C22 to C25, C2 to C3, C3 to C4, C4 to C5, C20 to C6, C5 to C7, C6 to C8, C7 to C9, IC1 to IC2, IC2 to IC4, R7 to R10, R9 to R11, R1 to R2, R3 to R4, R4 to R7, R5 to R8, R6 to R9, U4 to U3, U3 to U4, X2 to X1, X1 to X2
Connections:
- net labels added: PIEZO_A, PIEZO_B
- net labels removed: PIEZO, SYNC
- wire segments 224 -> 238
- no-connect marks 15 -> 18

Commit message: some routing improvements
Parts:
- added C26: 100n, control:C0603, symbol C
Connections:
- wire segments 238 -> 240

Commit message: update wifi, routing, gen gerbers, DONE r1
Parts:
- removed U2: ESP8266, control:ESP8266, symbol ESP8266
- added U2: ESP8266-ESP01, control:ESP8266-ESP01, symbol ESP8266-ESP01
Connections:
- net labels added: WIFI_GP0, WIFI_RST
- wire segments 240 -> 243
- no-connect marks 18 -> 17
Other:
- note added: "+5V from USB here so can\nbe shorted to VCC for development,\nleave NC on power board"
- note removed: "+5V from USB here so can be shorted to\nVCC for development, leave NC on power board"

Commit message: fix a few derps, actually DONE r1
Parts:
- CON1: Farnell 2443120 -> 2443111

Commit message: add resistor to red LED, closes #4
Parts:
- added R?: 50R, control:R0603, symbol R-RESCUE-control
- C1, C10, C11, C12, C13, C14, C15, C16, C17, C18, C19, C2, C20, C21, C22, C23, C24, C25, C26, C3, C4, C5, C6, C7, C8, C9: symbol C -> C-RESCUE-control
- R1, R10, R11, R2, R3, R4, R5, R6, R7, R8, R9: symbol R -> R-RESCUE-control
Connections:
- wire segments 243 -> 246
Changed lines of the file:
@@
 EESchema Schematic File Version 2
+LIBS:control-rescue
 LIBS:power
 LIBS:device
@@
 LIBS:memory
 LIBS:xilinx
-LIBS:special
 LIBS:microcontrollers
 LIBS:dsp
@@
 $EndComp
 $Comp
-L R R8
+L R-RESCUE-control R8
 U 1 1 54D015F8
 P 1200 6350
@@
 $EndComp
 $Comp
-L R R10
+L R-RESCUE-control R10
 U 1 1 54D01636
 P 1200 6550
@@
 $EndComp
 $Comp
-L C C23
+L C-RESCUE-control C23
 U 1 1 54D01666
 P 1700 6450
@@
 $EndComp
 $Comp
-L C C22
+L C-RESCUE-control C22
 U 1 1 54D0169F
 P 1700 5950
@@
 $EndComp
 $Comp
-L C C25
+L C-RESCUE-control C25
 U 1 1 54D016D3
 P 1700 6950
@@
 $EndComp
 $Comp
-L R R11
+L R-RESCUE-control R11
 U 1 1 54D0171F
 P 2050 7000
@@
 $EndComp
 $Comp
-L C C16
+L C-RESCUE-control C16
 U 1 1 54D0178D
 P 2850 5750
@@
 $EndComp
 $Comp
-L C C17
+L C-RESCUE-control C17
 U 1 1 54D017E2
 P 3150 5750
@@
 $EndComp
 $Comp
-L R R9
+L R-RESCUE-control R9
 U 1 1 54D032F8
 P 3700 6450
@@
 $EndComp
 $Comp
-L C C24
+L C-RESCUE-control C24
 U 1 1 54D033E8
 P 4050 6700
@@
 $EndComp
 $Comp
-L C C4
+L C-RESCUE-control C4
 U 1 1 54D055AB
 P 1200 1600
@@
 $EndComp
 $Comp
-L C C5
+L C-RESCUE-control C5
 U 1 1 54D0579F
 P 1400 1600
@@
 $EndComp
 $Comp
-L C C8
+L C-RESCUE-control C8
 U 1 1 54D057CF
 P 2000 1600
@@
 $EndComp
 $Comp
-L C C9
+L C-RESCUE-control C9
 U 1 1 54D05800
 P 2200 1600
@@
 $EndComp
 $Comp
-L C C10
+L C-RESCUE-control C10
 U 1 1 54D064F7
 P 1950 2350
@@
 $EndComp
 $Comp
-L C C14
+L C-RESCUE-control C14
 U 1 1 54D06F5C
 P 1150 4250
@@
 $EndComp
 $Comp
-L C C15
+L C-RESCUE-control C15
 U 1 1 54D06FE0
 P 1850 4250
@@
 $EndComp
 $Comp
-L R R7
+L R-RESCUE-control R7
 U 1 1 54D0713C
 P 1850 3450
@@
 	1    0    0    -1
 $EndComp
-Text Label 6850 1150 2    60   ~ 0
+Text Label 6950 800  2    60   ~ 0
 ENC_RED
 Text Label 6850 1250 2    60   ~ 0
@@
 +5V from USB here so can\nbe shorted to VCC for development,\nleave NC on power board
 $Comp
-L C C3
+L C-RESCUE-control C3
 U 1 1 54D1D963
 P 1000 1600
@@
 $EndComp
 $Comp
-L C C7
+L C-RESCUE-control C7
 U 1 1 54D1E2D0
 P 1800 1600
@@
 $EndComp
 $Comp
-L C C18
+L C-RESCUE-control C18
 U 1 1 54D25C39
 P 5700 5800
@@
 $EndComp
 $Comp
-L C C19
+L C-RESCUE-control C19
 U 1 1 54D25D98
 P 6950 5800
@@
 $EndComp
 $Comp
-L C C20
+L C-RESCUE-control C20
 U 1 1 54D25FC3
 P 7200 5800
@@
 $EndComp
 $Comp
-L C C21
+L C-RESCUE-control C21
 U 1 1 54D26038
 P 7450 5800
@@
 VOLTAGE REGULATION
 $Comp
-L R R2
+L R-RESCUE-control R2
 U 1 1 54D298B1
 P 7850 850
@@
 $EndComp
 $Comp
-L R R4
+L R-RESCUE-control R4
 U 1 1 54D29E22
 P 7850 1650
@@
 $EndComp
 $Comp
-L C C2
+L C-RESCUE-control C2
 U 1 1 54D29F7C
 P 8200 1450
@@
 $EndComp
 $Comp
-L C C1
+L C-RESCUE-control C1
 U 1 1 54D2A0F2
 P 8200 1000
@@
 $EndComp
 $Comp
-L C C12
+L C-RESCUE-control C12
 U 1 1 54D575FE
 P 1000 3150
@@
 $EndComp
 $Comp
-L C C11
+L C-RESCUE-control C11
 U 1 1 54D57653
 P 1000 2450
@@
 ~OLED_RST
 $Comp
-L C C13
+L C-RESCUE-control C13
 U 1 1 54DF5EF1
 P 9650 4100
@@
 NoConn ~ 3800 3350
 $Comp
-L C C6
+L C-RESCUE-control C6
 U 1 1 54E8BB79
 P 1600 1600
@@
 $EndComp
 $Comp
-L R R3
+L R-RESCUE-control R3
 U 1 1 54F54B30
 P 9400 1300
@@
 $EndComp
 $Comp
-L R R6
+L R-RESCUE-control R6
 U 1 1 54F54B8D
 P 9400 2350
@@
 $EndComp
 $Comp
-L R R1
+L R-RESCUE-control R1
 U 1 1 54F54D54
 P 9950 800
@@
 $EndComp
 $Comp
-L R R5
+L R-RESCUE-control R5
 U 1 1 54F56093
 P 9950 2050
@@
 NoConn ~ 2500 3450
 $Comp
-L C C26
+L C-RESCUE-control C26
 U 1 1 54F78010
 P 10650 1000
@@
 	6850 1250 6950 1250
 Wire Wire Line
-	6850 1150 6950 1150
+	6500 1150 6950 1150
 Wire Wire Line
 	6850 1550 6950 1550
@@
 Wire Wire Line
 	10150 4100 10000 4100
+$Comp
+L R-RESCUE-control R?
+U 1 1 56116BC9
+P 6750 950
+F 0 "R?" V 6830 950 50  0000 C CNN
+F 1 "50R" V 6757 951 50  0000 C CNN
+F 2 "control:R0603" V 6680 950 30  0001 C CNN
+F 3 "" H 6750 950 30  0000 C CNN
+F 4 "2331983" H 6750 950 60  0001 C CNN "Farnell"
+	1    6750 950
+	0    1    1    0
+$EndComp
+Wire Wire Line
+	6950 800  7000 800
+Wire Wire Line
+	7000 800  7000 950
+Wire Wire Line
+	6500 1150 6500 950
 $EndSCHEMATC
