File: control/control.sch (KiCad schematic (older format))
At the start: 60 parts, among them CON1 USB-MICRO-B, IC1 AD8542, IC2 STM32F072CBT6, IC3 ADP3335, IC4 AD8495, P1 SWD, P2 CONN_02X04, P3 CONN_01X02, U1 ROTENC, U2 ESP8266-ESP01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

Commit message: add ldo for wifi, closes #7 probably
Parts:
- added C27, C28: 10µ, control:C0603, symbol C-RESCUE-control
- added IC5: NCP1117, control:SOT223, symbol NCP1117
- gave numbers to parts that had none: 1
Connections:
- wire segments 246 -> 258

Commit message: smaller 32k xtal, closes #21
Parts:
- X1: footprint control:SMD_XTAL_8038 -> control:R0805; Farnell 2308714 -> 2467860
Changed lines of the file:
@@
 F 0 "X1" H 1400 2950 50  0000 C CNN
 F 1 "32k768" H 1400 2650 50  0000 C CNN
-F 2 "control:SMD_XTAL_8038" H 1400 2800 60  0001 C CNN
+F 2 "control:R0805" H 1400 2800 60  0001 C CNN
 F 3 "" H 1400 2800 60  0000 C CNN
-F 4 "2308714" H 1400 2800 60  0001 C CNN "Farnell"
+F 4 "2467860" H 1400 2800 60  0001 C CNN "Farnell"
 	1    1400 2800
 	0    1    1    0

Commit message: add LEDs to control, closes #22
Parts:
- added D?: GRN, control:LED0603, symbol Led_Small
- added D?: BLU, control:LED0603, symbol Led_Small
- added R? (x2): 1k, control:R0603, symbol R_Small
Connections:
- wire segments 258 -> 265
- no-connect marks 17 -> 15
Changed lines of the file:
@@
 OLED_MOSI
 NoConn ~ 3800 2650
-NoConn ~ 3800 3150
-NoConn ~ 3800 3250
 NoConn ~ 3800 3350
 $Comp
@@
 Wire Wire Line
 	6150 3100 6150 3150
+$Comp
+L Led_Small D?
+U 1 1 56117821
+P 4200 3150
+F 0 "D?" H 4150 3275 50  0000 L CNN
+F 1 "GRN" H 4100 3050 50  0000 L CNN
+F 2 "control:LED0603" V 4200 3150 60  0001 C CNN
+F 3 "" V 4200 3150 60  0000 C CNN
+F 4 "2290328" H 4200 3150 60  0001 C CNN "Farnell"
+	1    4200 3150
+	-1   0    0    1
+$EndComp
+$Comp
+L Led_Small D?
+U 1 1 56117AA6
+P 4200 3250
+F 0 "D?" H 4150 3375 50  0000 L CNN
+F 1 "BLU" H 4100 3150 50  0000 L CNN
+F 2 "control:LED0603" V 4200 3250 60  0001 C CNN
+F 3 "" V 4200 3250 60  0000 C CNN
+F 4 "2217972" H 4200 3250 60  0001 C CNN "Farnell"
+	1    4200 3250
+	-1   0    0    1
+$EndComp
+$Comp
+L R_Small R?
+U 1 1 56117B3C
+P 3950 3150
+F 0 "R?" H 3980 3170 50  0000 L CNN
+F 1 "1k" H 3980 3110 50  0000 L CNN
+F 2 "control:R0603" H 3950 3150 60  0001 C CNN
+F 3 "" H 3950 3150 60  0000 C CNN
+F 4 "2332003" H 3950 3150 60  0001 C CNN "Farnell"
+	1    3950 3150
+	0    1    1    0
+$EndComp
+$Comp
+L R_Small R?
+U 1 1 56117F84
+P 3950 3250
+F 0 "R?" H 3980 3270 50  0000 L CNN
+F 1 "1k" H 3980 3210 50  0000 L CNN
+F 2 "control:R0603" H 3950 3250 60  0001 C CNN
+F 3 "" H 3950 3250 60  0000 C CNN
+F 4 "2332003" H 3950 3250 60  0001 C CNN "Farnell"
+	1    3950 3250
+	0    1    1    0
+$EndComp
+$Comp
+L GND #PWR?
+U 1 1 5611876B
+P 4400 3300
+F 0 "#PWR?" H 4400 3050 60  0001 C CNN
+F 1 "GND" H 4400 3150 60  0000 C CNN
+F 2 "" H 4400 3300 60  0000 C CNN
+F 3 "" H 4400 3300 60  0000 C CNN
+	1    4400 3300
+	1    0    0    -1
+$EndComp
+Wire Wire Line
+	3800 3150 3850 3150
+Wire Wire Line
+	3800 3250 3850 3250
+Wire Wire Line
+	4050 3150 4100 3150
+Wire Wire Line
+	4050 3250 4100 3250
+Wire Wire Line
+	4300 3150 4400 3150
+Wire Wire Line
+	4400 3150 4400 3300
+Wire Wire Line
+	4300 3250 4400 3250
+Connection ~ 4400 3250
 $EndSCHEMATC

Commit message: add more resistors to rot end LEDs
Parts:
- added R15, R16: 50R, control:R0603, symbol R_Small
- R12: symbol R-RESCUE-control -> R_Small
- gave numbers to parts that had none: 4
Connections:
- wire segments 265 -> 264

Commit message: add tagconnect TC2030-CTX-NL footprint
Parts:
- added P?: CONN_02X03, control:TC2030-NL, symbol CONN_02X03
Connections:
- no-connect marks 15 -> 16
Changed lines of the file:
@@
 L SWD P1
 U 1 1 54CFFE52
-P 5350 1300
-F 0 "P1" H 5600 1600 60  0000 C CNN
-F 1 "SWD" H 5050 1600 60  0000 C CNN
-F 2 "control:FTSH-105-01-F-D-K" H 5700 1100 60  0001 C CNN
-F 3 "" H 5700 1100 60  0000 C CNN
-F 4 "1667759" H 5350 1300 60  0001 C CNN "Farnell"
-	1    5350 1300
+P 5300 1000
+F 0 "P1" H 5550 1300 60  0000 C CNN
+F 1 "SWD" H 5000 1300 60  0000 C CNN
+F 2 "control:FTSH-105-01-F-D-K" H 5650 800 60  0001 C CNN
+F 3 "" H 5650 800 60  0000 C CNN
+F 4 "1667759" H 5300 1000 60  0001 C CNN "Farnell"
+	1    5300 1000
 	1    0    0    -1
 $EndComp
@@
 L VDD #PWR4
 U 1 1 54D0D617
-P 4800 1050
-F 0 "#PWR4" H 4800 900 60  0001 C CNN
-F 1 "VDD" H 4800 1200 60  0000 C CNN
-F 2 "" H 4800 1050 60  0000 C CNN
-F 3 "" H 4800 1050 60  0000 C CNN
-	1    4800 1050
+P 4750 750
+F 0 "#PWR4" H 4750 600 60  0001 C CNN
+F 1 "VDD" H 4750 900 60  0000 C CNN
+F 2 "" H 4750 750 60  0000 C CNN
+F 3 "" H 4750 750 60  0000 C CNN
+	1    4750 750
 	1    0    0    -1
 $EndComp
@@
 L GND #PWR9
 U 1 1 54D11313
-P 4800 1550
-F 0 "#PWR9" H 4800 1300 60  0001 C CNN
-F 1 "GND" H 4800 1400 60  0000 C CNN
-F 2 "" H 4800 1550 60  0000 C CNN
-F 3 "" H 4800 1550 60  0000 C CNN
-	1    4800 1550
-	1    0    0    -1
-$EndComp
-Text Label 5900 1500 0    60   ~ 0
+P 4750 1250
+F 0 "#PWR9" H 4750 1000 60  0001 C CNN
+F 1 "GND" H 4750 1100 60  0000 C CNN
+F 2 "" H 4750 1250 60  0000 C CNN
+F 3 "" H 4750 1250 60  0000 C CNN
+	1    4750 1250
+	1    0    0    -1
+$EndComp
+Text Label 5850 1200 0    60   ~ 0
 nRST
-Text Label 5900 1200 0    60   ~ 0
+Text Label 5850 900  0    60   ~ 0
 SWDCLK
-Text Label 5900 1100 0    60   ~ 0
+Text Label 5850 800  0    60   ~ 0
 SWDIO
-NoConn ~ 5800 1300
-NoConn ~ 5800 1400
+NoConn ~ 5750 1000
+NoConn ~ 5750 1100
 Text Label 3900 1850 0    60   ~ 0
 SWDIO
@@
 	3900 1950 3800 1950
 Wire Wire Line
-	5800 1100 5900 1100
-Wire Wire Line
-	5800 1200 5900 1200
-Wire Wire Line
-	5800 1500 5900 1500
-Connection ~ 4800 1300
-Wire Wire Line
-	4850 1200 4800 1200
-Connection ~ 4800 1500
-Wire Wire Line
-	4850 1300 4800 1300
-Wire Wire Line
-	4800 1200 4800 1550
-Wire Wire Line
-	4800 1500 4850 1500
+	5750 800  5850 800
+Wire Wire Line
+	5750 900  5850 900
+Wire Wire Line
+	5750 1200 5850 1200
+Connection ~ 4750 1000
+Wire Wire Line
+	4800 900  4750 900
+Connection ~ 4750 1200
+Wire Wire Line
+	4800 1000 4750 1000
+Wire Wire Line
+	4750 900  4750 1250
+Wire Wire Line
+	4750 1200 4800 1200
 Wire Wire Line
 	7900 3900 8050 3900
@@
 	6850 3800 7400 3800
 Wire Wire Line
-	4800 1100 4850 1100
-Wire Wire Line
-	4800 1050 4800 1100
+	4750 800  4800 800
+Wire Wire Line
+	4750 750  4750 800
 Connection ~ 3150 5500
 Wire Wire Line
@@
 Wire Wire Line
 	6550 1350 6750 1350
+$Comp
+L CONN_02X03 P?
+U 1 1 561193DD
+P 5600 1700
+F 0 "P?" H 5600 1900 50  0000 C CNN
+F 1 "CONN_02X03" H 5600 1500 50  0000 C CNN
+F 2 "control:TC2030-NL" H 5600 500 60  0001 C CNN
+F 3 "" H 5600 500 60  0000 C CNN
+	1    5600 1700
+	1    0    0    -1
+$EndComp
+$Comp
+L VDD #PWR?
+U 1 1 5611983A
+P 5350 1600
+F 0 "#PWR?" H 5350 1450 60  0001 C CNN
+F 1 "VDD" H 5350 1750 60  0000 C CNN
+F 2 "" H 5350 1600 60  0000 C CNN
+F 3 "" H 5350 1600 60  0000 C CNN
+	1    5350 1600
+	1    0    0    -1
+$EndComp
+$Comp
+L GND #PWR?
+U 1 1 56119A7D
+P 5350 1800
+F 0 "#PWR?" H 5350 1550 60  0001 C CNN
+F 1 "GND" H 5350 1650 60  0000 C CNN
+F 2 "" H 5350 1800 60  0000 C CNN
+F 3 "" H 5350 1800 60  0000 C CNN
+	1    5350 1800
+	1    0    0    -1
+$EndComp
+Text Label 5850 1600 0    60   ~ 0
+SWDIO
+Text Label 5350 1700 2    60   ~ 0
+nRST
+Text Label 5850 1700 0    60   ~ 0
+SWDCLK
+NoConn ~ 5850 1800
 $EndSCHEMATC

Commit message: rework buzzer driver to use non-inverting amplifiers
Parts:
- added D5: CGA0402MLC-12G, control:R0402, symbol CGA0402MLC-12G
- R1, R5: value 15k -> 4k7; Farnell 2332018 -> 2332011
- gave numbers to parts that had none: 1
Connections:
- wire segments 264 -> 270
Other:
- moved on the sheet: R1, R3, R5, R6

Commit message: bom update
Parts:
- R13, R14: Farnell 2332003 -> 2116678
Changed lines of the file:
@@
 F 2 "control:R0603" H 3950 3150 60  0001 C CNN
 F 3 "" H 3950 3150 60  0000 C CNN
-F 4 "2332003" H 3950 3150 60  0001 C CNN "Farnell"
+F 4 "2116678" H 3950 3150 60  0001 C CNN "Farnell"
 	1    3950 3150
 	0    1    1    0
@@
 F 2 "control:R0603" H 3950 3250 60  0001 C CNN
 F 3 "" H 3950 3250 60  0000 C CNN
-F 4 "2332003" H 3950 3250 60  0001 C CNN "Farnell"
+F 4 "2116678" H 3950 3250 60  0001 C CNN "Farnell"
 	1    3950 3250
 	0    1    1    0
