File: control/control.kicad_pcb (KiCad board)
At the start: 2 copper layers, 100 x 40 mm, 60 parts, among them CON1 USB-MICRO-B, IC1 AD8542, IC2 STM32F072CBT6, IC3 ADP3335, IC4 AD8495, P1 SWD, P2 CONN_02X04, P3 CONN_01X02, U1 ROTENC, U2 ESP8266-ESP01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

Commit message: add ldo for wifi, closes #7 probably
Parts:
- added C27: 10µ, control:C0603, B.Cu at (68.0, 125.0)
- added C28: 10µ, control:C0603, B.Cu at (70.0, 125.0)
- added IC5: NCP1117, control:SOT223, B.Cu at (70.0, 122.5)
Connections:
- U2 pad 6: VDD -> Net-(C28-Pad1)
- U2 pad 8: VDD -> Net-(C28-Pad1)
Routing:
- net Net-(C28-Pad1): track 0.00 -> 29.2 mm
- net VDD: track 315.9 -> 301.8 mm
- net VCC: track 72.8 -> 84.4 mm, vias 0 -> 2
- net GND: track 68.7 -> 71.9 mm, vias 19 -> 21
